Commit message: added upper body to lower body. i changed some lower body configurations including removing the two base links in the legs and added a single pelvis link. i moved the intertial macro to a new utilities file

File: robotv1_description/urdf/robotv1.xacro (robot description, xacro)
@@ -2,300 +2,27 @@
 <!-- Revolute-Revolute Manipulator -->
 <robot name="robotv1" xmlns:xacro="http://www.ros.org/wiki/xacro" >
-  <!--Constant for the robotv1-->
-  <xacro:property name="Pi" value="3.1415926535897931"/>
-  <xacro:property name="density" value="2700"/>
-  <xacro:property name="lenx_base" value="0.06"/>
-  <xacro:property name="leny_base" value="0.08"/>
-  <xacro:property name="lenz_base" value="0.03"/>
-  <xacro:property name="lenx_hip_2" value="0.04"/>
-  <xacro:property name="leny_hip_2" value="0.03"/>
-  <xacro:property name="lenz_hip_2" value="0.06"/>
-  <xacro:property name="lenx_hip_3" value="0.07"/>
-  <xacro:property name="leny_hip_3" value="0.03"/>
-  <xacro:property name="lenz_hip_3" value="0.09"/>
-  <xacro:property name="lenx_upp" value="0.03"/>
-  <xacro:property name="leny_upp" value="0.04"/>
-  <xacro:property name="lenz_upp" value="0.06"/>
-  <xacro:property name="lenx_low" value="0.02"/>
-  <xacro:property name="leny_low" value="0.02"/>
-  <xacro:property name="lenz_low" value="0.14"/>
-  <xacro:property name="lenx_ang_1" value="0.04"/>
-  <xacro:property name="leny_ang_1" value="0.03"/>
-  <xacro:property name="lenz_ang_1" value="0.06"/>
-  <xacro:property name="lenx_ang_2" value="0.03"/>
-  <xacro:property name="leny_ang_2" value="0.04"/>
-  <xacro:property name="lenz_ang_2" value="0.06"/>
-  <xacro:property name="lenx_foot" value="0.1"/>
-  <xacro:property name="leny_foot" value="0.04"/>
-  <xacro:property name="lenz_foot" value="0.002"/>
-  <xacro:property name="mass_base" value="${density*lenx_base*leny_base*lenz_base}"/>
-  <xacro:property name="mass_hip_2" value="${density*lenx_hip_2*leny_hip_2*lenz_hip_2}"/>
-  <xacro:property name="mass_hip_3" value="${density*lenx_hip_3*leny_hip_3*lenz_hip_3}"/>
-  <xacro:property name="mass_upp" value="${density*lenx_upp*leny_upp*lenz_upp}"/>
-  <xacro:property name="mass_low" value="${density*lenx_low*leny_low*lenz_low}"/>
-  <xacro:property name="mass_ang_1" value="${density*lenx_ang_1*leny_ang_1*lenz_ang_1}"/>
-  <xacro:property name="mass_ang_2" value="${density*lenx_ang_2*leny_ang_2*lenz_ang_2}"/>
-  <xacro:property name="mass_foot" value="${density*lenx_foot*leny_foot*lenz_foot}"/>
-  <xacro:include filename="$(find robotv1_description)/materials/materials.xacro" />
-  <xacro:include filename="$(find robotv1_description)/urdf/robotv1.gazebo" />
-  <xacro:macro name="box_inertia" params="mass lenx leny lenz">
+  <xacro:include filename="$(find robotv1_description)/urdf/lower_body.xacro"/>
+  <xacro:include filename="$(find robotv1_description)/urdf/upper_body.xacro"/>
+  <link name="world">
     <inertial>
-      <mass value="${mass}" />
+      <origin xyz="0 0 1" rpy="0 0 0"/>
+      <mass value="1"/>
       <inertia
-      ixx="${100*mass*(lenz*lenz+leny*leny)/12}" ixy="0.0" ixz="0.0"
-      iyy="${100*mass*(lenz*lenz+leny*leny)/12}" iyz="0.0"
-      izz="${100*mass*(lenz*lenz+leny*leny)/12}" />
+        ixx="1.0" ixy="0.0" ixz="0.0"
+        iyy="1.0" iyz="0.0"
+        izz="1.0"/>
     </inertial>
-  </xacro:macro>
-  <xacro:macro name="leg" params="prefix reflect" >
-    <joint name="${prefix}_hip_1_joint" type="revolute" >
-      <parent link="base"/>
-      <child link="${prefix}_hip_2"/>
-      <origin xyz="0 ${leny_base*reflect/2} 0"/>
-      <axis xyz="0 1 0"/>
-      <dynamics damping="0.7"/>
-      <limit effort="20" velocity="1.0" lower="${-Pi/2}" upper="${Pi/2}" />
-    </joint>
-    <link name="${prefix}_hip_2" >
-      <visual>
-        <origin xyz="0 ${leny_hip_2*reflect/2} 0" rpy="0 0 0"/>
-        <geometry>
-          <box size="${lenx_hip_2} ${leny_hip_2} ${lenz_hip_2}"/>
-        </geometry>
-        <material name="black"/>
-      </visual>
-      <xacro:box_inertia mass="${mass_hip_2}" lenx="${lenx_hip_2}" leny="${leny_hip_2}" lenz="${lenz_hip_2}" />
-      <collision>
-        <origin xyz="0 ${leny_hip_2*reflect/2} 0" rpy="0 0 0"/>
-        <geometry>
-          <box size="${lenx_hip_2} ${leny_hip_2} ${lenz_hip_2}"/>
-        </geometry>
-     </collision>
-   </link>
-   <joint name="${prefix}_hip_2_joint" type="revolute" >
-      <parent link="${prefix}_hip_2"/>
-      <child link="${prefix}_hip_3"/>
-      <origin xyz= "0 ${leny_hip_2*reflect} 0"/>
-      <axis xyz="1 0 0"/>
-      <dynamics damping="0.7"/>
-      <limit effort="20" velocity="1.0" lower="${-Pi/2}" upper="${Pi/2}" />
-    </joint>
-    <link name="${prefix}_hip_3" >
-      <visual>
-        <origin xyz="0 0 ${-1*lenz_hip_3/2 }" rpy="0 0 0"/>
-        <geometry>
-          <box size="${lenx_hip_3} ${leny_hip_3} ${lenz_hip_3}"/>
-        </geometry>
-        <material name="orange"/>
-      </visual>
-     <xacro:box_inertia mass="${mass_hip_3}" lenx="${lenx_hip_3}" leny="${leny_hip_3}" lenz="${lenz_hip_3}" />
-     <collision>
-        <origin xyz="0 0 ${-1*lenz_hip_3/2 }" rpy="0 0 0"/>
-        <geometry>
-          <box size="${lenx_hip_3} ${leny_hip_3} ${lenz_hip_3}"/>
-        </geometry>
-     </collision>
-    </link>
-    <joint name="${prefix}_hip_3_joint" type="revolute" >
-      <parent link="${prefix}_hip_3"/>
-      <child link="${prefix}_upp"/>
-      <origin xyz="0 0 ${-1*lenz_hip_3 }"/>
-      <axis xyz="0 0 1"/>
-      <dynamics damping="0.7"/>
-      <limit effort="20" velocity="1.0" lower="${-Pi/2}" upper="${Pi/2}" />
-    </joint>
-    <link name="${prefix}_upp" >
-      <visual>
-        <origin xyz="0 0 ${-1*lenz_upp/2}" rpy="0 0 0"/>
-        <geometry>
-          <box size="${lenx_upp} ${leny_upp} ${lenz_upp}"/>
-        </geometry>
-        <material name="black"/>
-      </visual>
-     <xacro:box_inertia mass="${mass_upp}" lenx="${lenx_upp}" leny="${leny_upp}" lenz="${lenz_upp}" />
-     <collision>
-        <origin xyz="0 0 ${-1*lenz_upp/2}" rpy="0 0 0"/>
-        <geometry>
-          <box size="${lenx_upp} ${leny_upp} ${lenz_upp}"/>
-        </geometry>
-     </collision>
-    </link>
-    <joint name="${prefix}_knee_joint" type="revolute" >
-      <parent link="${prefix}_upp"/>
-      <child link="${prefix}_low"/>
-      <origin xyz="0 0 ${-lenz_upp}"/>
-      <axis xyz="0 1 0"/>
-      <dynamics damping="0.7"/>
-      <limit effort="20" velocity="1.0" lower="0" upper="${7*Pi/8}" />
-    </joint>
-    <link name="${prefix}_low" >
-      <visual>
-        <origin xyz="0 0 ${-lenz_low/2}" rpy="0 0 0"/>
-        <geometry>
-         <box size="${lenx_low} ${leny_low} ${lenz_low}"/>
-        </geometry>
-        <material name="orange"/>
-      </visual>
-     <xacro:box_inertia mass="${mass_low}" lenx="${lenx_low}" leny="${leny_low}" lenz="${lenz_low}" />
-     <collision>
-       <origin xyz="0 0 ${-lenz_low/2}" rpy="0 0 0"/>
-       <geometry>
-         <box size="${lenx_low} ${leny_low} ${lenz_low}"/>
-       </geometry>
-     </collision>
-    </link>
-    <joint name="${prefix}_ang_1_joint" type="revolute" >
-      <parent link="${prefix}_low"/>
-      <child link="${prefix}_ang_1"/>
-      <origin xyz="0 0 ${-lenz_low+lenz_ang_1/2}" rpy="0 0 0"/>
-      <axis xyz="1 0 0"/>
-      <dynamics damping="0.7"/>
-      <limit effort="20" velocity="1.0" lower="${-Pi/4}" upper="${Pi/4}" />
-    </joint>
-    <link name="${prefix}_ang_1" >
-      <visual>
-      <origin xyz="0 0 0" rpy="0 0 0"/>
-        <geometry>
-          <box size="${lenx_ang_1} ${leny_ang_1} ${lenz_ang_1}"/>
-        </geometry>
-        <material name="black"/>
-      </visual>
-     <xacro:box_inertia mass="${mass_ang_1}" lenx="${lenx_ang_1}" leny="${leny_ang_1}" lenz="${lenz_ang_1}" />
-     <collision>
-       <origin xyz="0 0 0" rpy="0 0 0"/>
-       <geometry>
-         <box size="${lenx_ang_1} ${leny_ang_1} ${lenz_ang_1}"/>
-       </geometry>
-      </collision>
-     </link>
-     <joint name="${prefix}_ang_2_joint" type="revolute" >
-       <parent link="${prefix}_ang_1"/>
-       <child link="${prefix}_ang_2"/>
-       <origin xyz="${-lenx_ang_1/2} 0 0"/>
-       <axis xyz="0 1 0"/>
-       <dynamics damping="0.7"/>
-       <limit effort="20" velocity="1.0" lower="${-Pi/4}" upper="${Pi/4}" />
-     </joint>
-     <link name="${prefix}_ang_2" >
-       <visual>
-       <origin xyz="0 0 ${-lenz_ang_2/2}" rpy="0 0 0"/>
-         <geometry>
-           <box size="${lenx_ang_2} ${leny_ang_2} ${lenz_ang_2}"/>
-         </geometry>
-         <material name="orange"/>
-       </visual>
-     <xacro:box_inertia mass="${mass_ang_2}" lenx="${lenx_ang_2}" leny="${leny_ang_2}" lenz="${lenz_ang_2}" />
-      <collision>
-       <origin xyz="${-lenx_ang_1} 0 ${-lenz_ang_2/2}" rpy="0 0 0"/>
-        <geometry>
-          <box size="${lenx_ang_2} ${leny_ang_2} ${lenz_ang_2}"/>
-        </geometry>
-      </collision>
-    </link>
-    <joint name="${prefix}_foot_joint" type="fixed" >
-      <parent link="${prefix}_ang_2"/>
-      <child link="${prefix}_foot"/>
-      <origin xyz="0 0 ${-lenz_ang_2}"/>
-    </joint>
-    <link name="${prefix}_foot" >
-      <visual>
-        <origin xyz="${lenx_foot/2-lenx_ang_2/2} 0 ${-lenz_foot/2}" rpy="0 0 0"/>
-        <geometry>
-          <box size="${lenx_foot} ${leny_foot} ${lenz_foot}"/>
-        </geometry>
-        <material name="orange"/>
-      </visual>
-     <xacro:box_inertia mass="${mass_foot}" lenx="${lenx_foot}" leny="${leny_foot}" lenz="${lenz_foot}" />
-     <collision>
-       <origin xyz="${lenx_foot/2-lenx_ang_2/2} 0 ${-lenz_foot/2}" rpy="0 0 0"/>
-       <geometry>
-          <box size="${lenx_foot} ${leny_foot} ${lenz_foot}"/>
-       </geometry>
-     </collision>
-    </link>
-    <transmission name="${prefix}_hip_1_tran">
-      <type>transmission_interface/SimpleTransmission</type>
-      <joint name="${prefix}_hip_1_joint">
-        <hardwareInterface>hardware_interface/EffortJointInterface</hardwareInterface>
-      </joint>
-      <actuator name="${prefix}_hip_1_motor">
-        <hardwareInterface>hardware_interface/EffortJointInterface</hardwareInterface>
-        <mechanicalReduction>1</mechanicalReduction>
-      </actuator>
-    </transmission>
-    <transmission name="${prefix}_hip_2_tran">
-      <type>transmission_interface/SimpleTransmission</type>
-      <joint name="${prefix}_hip_2_joint">
-        <hardwareInterface>hardware_interface/EffortJointInterface</hardwareInterface>
-      </joint>
-      <actuator name="${prefix}_hip_2_motor">
-        <hardwareInterface>hardware_interface/EffortJointInterface</hardwareInterface>
-        <mechanicalReduction>1</mechanicalReduction>
-      </actuator>
-    </transmission>
-    <transmission name="${prefix}_hip_3_tran">
-      <type>transmission_interface/SimpleTransmission</type>
-      <joint name="${prefix}_hip_3_joint">
-        <hardwareInterface>hardware_interface/EffortJointInterface</hardwareInterface>
-      </joint>
-      <actuator name="${prefix}_hip_3_motor">
-        <hardwareInterface>hardware_interface/EffortJointInterface</hardwareInterface>
-        <mechanicalReduction>1</mechanicalReduction>
-      </actuator>
-    </transmission>
-    <transmission name="${prefix}_knee_tran">
-      <type>transmission_interface/SimpleTransmission</type>
-      <joint name="${prefix}_knee_joint">
-        <hardwareInterface>hardware_interface/EffortJointInterface</hardwareInterface>
-      </joint>
-      <actuator name="${prefix}_knee_motor">
-        <hardwareInterface>hardware_interface/EffortJointInterface</hardwareInterface>
-        <mechanicalReduction>1</mechanicalReduction>
-      </actuator>
-    </transmission>
-    <transmission name="${prefix}_ang_1_tran">
-      <type>transmission_interface/SimpleTransmission</type>
-      <joint name="${prefix}_ang_1_joint">
-        <hardwareInterface>hardware_interface/EffortJointInterface</hardwareInterface>
-      </joint>
-      <actuator name="${prefix}_ang_1_motor">
-        <hardwareInterface>hardware_interface/EffortJointInterface</hardwareInterface>
-        <mechanicalReduction>1</mechanicalReduction>
-      </actuator>
-    </transmission>
-    <transmission name="${prefix}_ang_2_tran">
-      <type>transmission_interface/SimpleTransmission</type>
-      <joint name="${prefix}_ang_2_joint">
-        <hardwareInterface>hardware_interface/EffortJointInterface</hardwareInterface>
-      </joint>
-      <actuator name="${prefix}_ang_2_motor">
-        <hardwareInterface>hardware_interface/EffortJointInterface</hardwareInterface>
-        <mechanicalReduction>1</mechanicalReduction>
-      </actuator>
-    </transmission>
- </xacro:macro>
- <link name="dummy"/>
-  <joint name="dummy_to_base" type="fixed" >
-    <parent link="dummy"/>
-    <child link="base"/>
-    <origin xyz="0 0 ${lenz_foot+lenz_ang_2-lenz_ang_1/2+lenz_low+lenz_upp+lenz_hip_3 }"/>
+  </link>
+  <joint name="fixed" type="fixed">
+    <parent link="world"/>
+    <child link="pelvis"/>
+    <origin xyz="0 0 1"/>
   </joint>
-  <link name="base" >
-    <visual>
-      <origin xyz="0 0 0 " rpy="0 0 0" />
-      <geometry>
-        <box size="${lenx_base} ${leny_base} ${lenz_base}"/>
-      </geometry>
-      <material name="orange"/>
-    </visual>
-    <xacro:box_inertia mass="${mass_base}" lenx="${lenx_base}" leny="${leny_base}" lenz="${lenz_base}"/>
-    <collision>
-      <origin xyz="0 0 0 " rpy="0 0 0" />
-      <geometry>
-        <box size="${lenx_base} ${leny_base} ${lenz_base}"/>
-      </geometry>
-    </collision>
-  </link>
-  <xacro:leg prefix="leftleg" reflect="1" />
-  <xacro:leg prefix="rightleg" reflect="-1" />
+  <joint name="pelvis_torso_joint" type="fixed">
+    <parent link="pelvis"/>
+    <child link="torso"/>
+    <origin xyz="0 0 ${lenz_pelvis/2}" rpy="0 0 0"/>
+    <axis xyz="0 1 0"/>
+    <limit lower="0" upper="${2*pi}" effort="${elbowEff}" velocity="${elbowVel}"/>
+  </joint>
 </robot>
