Commit message: updated robotv1 model

File: robotv1_description/urdf/arm.xacro (robot description, xacro)
@@ -1,50 +1,176 @@
 <?xml version="1.0"?>
-<robot name="arm" xmlns:xacro="http://www.ros.org/wiki/xacro">
+<robot xmlns:xacro="http://www.ros.org/wiki/xacro">
   <xacro:include filename="$(find robotv1_description)/urdf/utilities.xacro"/>
-  <xacro:property name="armWidth" value=".025"/>
-  <xacro:property name="upperArmLength" value="0.15"/>
-  <xacro:property name="lowerArmLength" value="0.07"/>
-  <xacro:property name="elbowEff" value="1.0"/>
-  <xacro:property name="elbowVel" value="1.0"/>
-  <xacro:macro name="robot_v1_arm" params="prefix reflect">
-    <link name="${prefix}_upper_arm">
-      <collision>
-        <origin xyz="0 0 ${upperArmLength/2}" rpy="0 0 0"/>
+  <xacro:include filename="$(find robotv1_description)/urdf/gripper.xacro"/>
+  <xacro:include filename="$(find robotv1_description)/urdf/arm.gazebo"/>
+  <xacro:property name="lenx_sho" value="0.06"/>
+  <xacro:property name="leny_sho" value="0.03"/>
+  <xacro:property name="lenz_sho" value="0.04"/>
+  <xacro:property name="lenx_upp_arm" value="0.02"/>
+  <xacro:property name="leny_upp_arm" value="0.06"/>
+  <xacro:property name="lenz_upp_arm" value="0.12"/>
+  <xacro:property name="lenx_low_arm" value="0.02"/>
+  <xacro:property name="leny_low_arm" value="0.04"/>
+  <xacro:property name="lenz_low_arm" value="0.07"/>
+  <xacro:property name="lenx_wri_1" value="0.04"/>
+  <xacro:property name="leny_wri_1" value="0.06"/>
+  <xacro:property name="lenz_wri_1" value="0.03"/>
+ <xacro:macro name="arm" params="prefix" >
+    <joint name="${prefix}_shoulder_1_joint" type="revolute" >
+      <parent link="pelvis"/>
+      <child link="${prefix}_sho"/>
+      <origin xyz="0 0 ${lenz_pelvis/2}"/>
+      <axis xyz="0 0 1"/>
+      <dynamics damping="0.7"/>
+      <limit effort="0.2" velocity="1.0" lower="${-pi/2}" upper="${pi/2}" />
+    </joint>
+    <link name="${prefix}_sho" >
+      <visual>
+        <origin xyz="0 0 ${lenz_sho/2}" rpy="0 0 0"/>
         <geometry>
-          <box size="${armWidth} ${armWidth} ${upperArmLength}"/>
-        </geometry>
-      </collision>
-      <visual>
-        <origin xyz="0 0 ${upperArmLength/2}" rpy="0 0 0"/>
-        <geometry>
-          <box size="${armWidth} ${armWidth} ${upperArmLength}"/>
-        </geometry>
-        <material name="orange"/>
-      </visual>
-        <xacro:box_inertia  lenx="${armWidth}" leny="${armWidth}" lenz="${upperArmLength}"/>
-    </link>
-    <link name="${prefix}_lower_arm">
-      <collision>
-        <origin xyz="0 0 ${lowerArmLength/2}" rpy="0 0 0"/>
-        <geometry>
-          <box size="${armWidth} ${armWidth} ${lowerArmLength}"/>
-        </geometry>
-      </collision>
-      <visual>
-        <origin xyz="0 0 ${lowerArmLength/2}" rpy="0 0 0"/>
-        <geometry>
-          <box size="${armWidth} ${armWidth} ${lowerArmLength}"/>
+          <box size="${lenx_sho} ${leny_sho} ${lenz_sho}"/>
         </geometry>
         <material name="black"/>
       </visual>
-      <xacro:box_inertia lenx="${armWidth}" leny="${armWidth}" lenz="${upperArmLength}"/>
-    </link>
-    <joint name="elbow" type="revolute">
-      <parent link="${prefix}_upper_arm"/>
-      <child link="${prefix}_lower_arm"/>
-      <origin xyz="0 0 ${upperArmLength}" rpy="0 0 0"/>
-      <axis xyz="0 1 0"/>
-      <limit lower="0" upper="${2*pi}" effort="${elbowEff}" velocity="${elbowVel}"/>
+      <xacro:box_inertia  lenx="${lenx_sho}" leny="${leny_sho}" lenz="${lenz_sho}" />
+      <collision>
+        <origin xyz="0 0 ${lenz_sho/2}" rpy="0 0 0"/>
+        <geometry>
+          <box size="${lenx_sho} ${leny_sho} ${lenz_sho}"/>
+        </geometry>
+     </collision>
+   </link>
+   <joint name="${prefix}_shoulder_2_joint" type="revolute" >
+     <parent link="${prefix}_sho"/>
+     <child link="${prefix}_upp_arm"/>
+     <origin xyz="0 0 ${lenz_sho/2}"/>
+     <axis xyz="0 1 0"/>
+     <dynamics damping="0.7"/>
+     <limit effort="0.2" velocity="1.0" lower="${-pi/2}" upper="${pi/2}" />
+   </joint>
+   <link name="${prefix}_upp_arm" >
+     <visual>
+       <origin xyz="0 0 ${lenz_upp_arm/2}" rpy="0 0 0"/>
+       <geometry>
+         <box size="${lenx_upp_arm} ${leny_upp_arm} ${lenz_upp_arm}"/>
+       </geometry>
+       <material name="orange"/>
+     </visual>
+     <xacro:box_inertia  lenx="${lenx_upp_arm}" leny="${leny_upp_arm}" lenz="${lenz_upp_arm}" />
+     <collision>
+       <origin xyz="0 0 ${lenz_upp_arm/2}" rpy="0 0 0"/>
+       <geometry>
+         <box size="${lenx_upp_arm} ${leny_upp_arm} ${lenz_upp_arm}"/>
+       </geometry>
+    </collision>
+  </link>
+  <joint name="${prefix}_elbow_joint" type="revolute" >
+    <parent link="${prefix}_upp_arm"/>
+    <child link="${prefix}_low_arm"/>
+    <origin xyz="0 0 ${lenz_upp_arm}"/>
+    <axis xyz="0 1 0"/>
+    <dynamics damping="0.7"/>
+    <limit effort="0.2" velocity="1.0" lower="0" upper="${pi}" />
+  </joint>
+  <link name="${prefix}_low_arm" >
+    <visual>
+      <origin xyz="0 0 ${lenz_low_arm/2}" rpy="0 0 0"/>
+      <geometry>
+        <box size="${lenx_low_arm} ${leny_low_arm} ${lenz_low_arm}"/>
+      </geometry>
+      <material name="black"/>
+    </visual>
+    <xacro:box_inertia  lenx="${lenx_low_arm}" leny="${leny_low_arm}" lenz="${lenz_low_arm}" />
+    <collision>
+      <origin xyz="0 0 ${lenz_low_arm/2}" rpy="0 0 0"/>
+      <geometry>
+        <box size="${lenx_low_arm} ${leny_low_arm} ${lenz_low_arm}"/>
+      </geometry>
+    </collision>
+  </link>
+  <joint name="${prefix}_wrist_1_joint" type="revolute" >
+    <parent link="${prefix}_low_arm"/>
+    <child link="${prefix}_wri_1"/>
+    <origin xyz="0 0 ${lenz_low_arm}"/>
+    <axis xyz="0 1 0"/>
+    <dynamics damping="0.7"/>
+    <limit effort="0.2" velocity="1.0" lower="${-pi/2}" upper="${pi/2}" />
+  </joint>
+  <link name="${prefix}_wri_1" >
+    <visual>
+      <origin xyz="0 0 ${lenz_wri_1/2}" rpy="0 0 0"/>
+      <geometry>
+        <box size="${lenx_wri_1} ${leny_wri_1} ${lenz_wri_1}"/>
+      </geometry>
+      <material name="orange"/>
+    </visual>
+    <xacro:box_inertia  lenx="${lenx_wri_1}" leny="${leny_wri_1}" lenz="${lenz_wri_1}" />
+    <collision>
+      <origin xyz="0 0 ${lenz_wri_1/2}" rpy="0 0 0"/>
+      <geometry>
+        <box size="${lenx_wri_1} ${leny_wri_1} ${lenz_wri_1}"/>
+      </geometry>
+    </collision>
+  </link>
+  <joint name="${prefix}_wrist_2_joint" type="revolute" >
+    <parent link="${prefix}_wri_1"/>
+    <child link="${prefix}_gripper"/>
+    <origin xyz="0 0 ${lenz_wri_1}"/>
+    <axis xyz="0 0 1"/>
+    <dynamics damping="0.7"/>
+    <limit effort="0.2" velocity="1.0" lower="${-pi/2}" upper="${pi/2}" />
+  </joint>
+  <xacro:gripper prefix="${prefix}"/>
+  <transmission name="${prefix}_shoulder_1_joint_tran">
+    <type> transmission_interface/SimpleTransmission</type>
+    <joint name="${prefix}_shoulder_1_joint">
+      <hardwareInterface>hardware_interface/EffortJointInterface</hardwareInterface>
     </joint>
-  </xacro:macro>
+    <actuator name="${prefix}_shoulder_1_joint_motor">
+      <hardwareInterface>hardware_interface/EffortJointInterface</hardwareInterface>
+      <mechanicalReduction>1</mechanicalReduction>
+    </actuator>
+  </transmission>
+  <transmission name="${prefix}_shoulder_2_joint_tran">
+    <type> transmission_interface/SimpleTransmission</type>
+    <joint name="${prefix}_shoulder_2_joint">
+      <hardwareInterface>hardware_interface/EffortJointInterface</hardwareInterface>
+    </joint>
+    <actuator name="${prefix}_shoulder_2_joint_motor">
+      <hardwareInterface>hardware_interface/EffortJointInterface</hardwareInterface>
+      <mechanicalReduction>1</mechanicalReduction>
+    </actuator>
+  </transmission>
+  <transmission name="${prefix}_elbow_joint_tran">
+    <type> transmission_interface/SimpleTransmission</type>
+    <joint name="${prefix}_elbow_joint">
+      <hardwareInterface>hardware_interface/EffortJointInterface</hardwareInterface>
+    </joint>
+    <actuator name="${prefix}_elbow_joint_motor">
+      <hardwareInterface>hardware_interface/EffortJointInterface</hardwareInterface>
+      <mechanicalReduction>1</mechanicalReduction>
+    </actuator>
+  </transmission>
+  <transmission name="${prefix}_wrist_1_joint_tran">
+    <type> transmission_interface/SimpleTransmission</type>
+    <joint name="${prefix}_wrist_1_joint">
+      <hardwareInterface>hardware_interface/EffortJointInterface</hardwareInterface>
+    </joint>
+    <actuator name="${prefix}_wrist_1_joint_motor">
+      <hardwareInterface>hardware_interface/EffortJointInterface</hardwareInterface>
+      <mechanicalReduction>1</mechanicalReduction>
+    </actuator>
+  </transmission>
+  <transmission name="${prefix}_wrist_2_joint_tran">
+    <type> transmission_interface/SimpleTransmission</type>
+    <joint name="${prefix}_wrist_2_joint">
+      <hardwareInterface>hardware_interface/EffortJointInterface</hardwareInterface>
+    </joint>
+    <actuator name="${prefix}_wrist_2_joint_motor">
+      <hardwareInterface>hardware_interface/EffortJointInterface</hardwareInterface>
+      <mechanicalReduction>1</mechanicalReduction>
+    </actuator>
+  </transmission>
+  <xacro:arm_gazebo_reference prefix="${prefix}"/>
+</xacro:macro>
 </robot>

File: robotv1_description/urdf/gripper.xacro (robot description, xacro)
@@ -1,22 +1,23 @@
 <?xml version="1.0"?>
-<robot xmlns:xacro="http://www.ros.org/wiki/xacro">
+<robot  xmlns:xacro="http://www.ros.org/wiki/xacro">
   <xacro:include filename="$(find robotv1_description)/urdf/utilities.xacro"/>
-  <xacro:property name="gripper_width" value="0.025"/>
-  <xacro:property name="gripper_length" value="0.025"/>
-  <xacro:macro name="robot_v1_gripper" params="prefix">
+  <xacro:property name="lenx_gri" value="0.06"/>
+  <xacro:property name="leny_gri" value="0.03"/>
+  <xacro:property name="lenz_gri" value="0.04"/>
+  <xacro:macro name="gripper" params="prefix">
     <link name="${prefix}_gripper">
       <visual>
         <geometry>
-          <box size="${gripper_width} ${gripper_width} ${gripper_length}"/>
+          <box size="${lenx_gri} ${leny_gri} ${lenz_gri}"/>
         </geometry>
       <origin rpy="0 0 0 " xyz="0.0 0 0"/>
-      <material name="orange"/>
+      <material name="black"/>
       </visual>
       <inertial>
-        <mass value="1"/>
+        <mass value=".01"/>
         <inertia
-          ixx="1.0" ixy="0.0" ixz="0.0"
-          iyy="1.0" iyz="0.0"
-          izz="1.0"/>
+          ixx="0.0001" ixy="0.0" ixz="0.0"
+          iyy="0.0001" iyz="0.0"
+          izz="0.0001"/>
       </inertial>
     </link>
@@ -26,9 +27,9 @@
       <child link="${prefix}_left_finger"/>
       <axis xyz="0 0 1"/>
-      <limit lower="0" upper="${pi}" effort="1" velocity="1"/>
+      <limit lower="0" upper="${pi/4}" effort="0.0001" velocity="0.0001"/>
     </joint>
     <link name="${prefix}_left_finger">
       <visual>
-      <origin rpy="0.0 0 0" xyz="0 0 0"/>
+      <origin rpy="0 0 0" xyz="0 0 0"/>
         <geometry>
           <mesh filename="package://urdf_tutorial/meshes/l_finger.dae"/>
@@ -36,9 +37,9 @@
       </visual>
       <inertial>
-        <mass value="1"/>
+        <mass value="0.01"/>
         <inertia
-          ixx="1.0" ixy="0.0" ixz="0.0"
-          iyy="1.0" iyz="0.0"
-          izz="1.0"/>
+          ixx="0.0001" ixy="0.0" ixz="0.0"
+          iyy="0.0001" iyz="0.0"
+          izz="0.0001"/>
       </inertial>
     </link>
@@ -55,9 +56,9 @@
       </visual>
       <inertial>
-        <mass value="1"/>
+        <mass value="0.01"/>
         <inertia
-          ixx="1.0" ixy="0.0" ixz="0.0"
-          iyy="1.0" iyz="0.0"
-          izz="1.0"/>
+          ixx="0.0001" ixy="0.0" ixz="0.0"
+          iyy="0.0001" iyz="0.0"
+          izz="0.0001"/>
       </inertial>
     </link>
@@ -67,5 +68,5 @@
       <child link="${prefix}_right_finger"/>
       <axis xyz="0 0 1"/>
-      <limit lower="0" upper="${pi}" effort="1" velocity="1"/>
+      <limit lower="${-pi/4}" upper="0" effort="0.0001" velocity="0.0001"/>
     </joint>
     <link name="${prefix}_right_finger">
@@ -77,9 +78,9 @@
     </visual>
       <inertial>
-        <mass value="1"/>
+        <mass value="0.01"/>
         <inertia
-          ixx="1.0" ixy="0.0" ixz="0.0"
-          iyy="1.0" iyz="0.0"
-          izz="1.0"/>
+          ixx="0.0001" ixy="0.0" ixz="0.0"
+          iyy="0.0001" iyz="0.0"
+          izz="0.0001"/>
       </inertial>
     </link>
@@ -96,11 +97,31 @@
       </visual>
       <inertial>
-        <mass value="1"/>
+        <mass value="0.01"/>
         <inertia
-          ixx="1.0" ixy="0.0" ixz="0.0"
-          iyy="1.0" iyz="0.0"
-          izz="1.0"/>
+          ixx="0.0001" ixy="0.0" ixz="0.0"
+          iyy="0.0001" iyz="0.0"
+          izz="0.0001"/>
       </inertial>
     </link>
+  <transmission name="${prefix}_left_finger_joint_tran">
+    <type> transmission_interface/SimpleTransmission</type>
+    <joint name="${prefix}_left_finger_joint">
+      <hardwareInterface>hardware_interface/EffortJointInterface</hardwareInterface>
+    </joint>
+    <actuator name="${prefix}_left_finger_joint_motor">
+      <hardwareInterface>hardware_interface/EffortJointInterface</hardwareInterface>
+      <mechanicalReduction>1</mechanicalReduction>
+    </actuator>
+  </transmission>
+  <transmission name="${prefix}_right_finger_joint_tran">
+    <type> transmission_interface/SimpleTransmission</type>
+    <joint name="${prefix}_right_finger_joint">
+      <hardwareInterface>hardware_interface/EffortJointInterface</hardwareInterface>
+    </joint>
+    <actuator name="${prefix}_right_finger_joint_motor">
+      <hardwareInterface>hardware_interface/EffortJointInterface</hardwareInterface>
+      <mechanicalReduction>1</mechanicalReduction>
+    </actuator>
+  </transmission>
   </xacro:macro>
 </robot>

File: robotv1_description/urdf/leg.xacro (robot description, xacro)
@@ -1,7 +1,6 @@
 <?xml version="1.0"?>
 <!-- Revolute-Revolute Manipulator -->
-<robot name="robotv1" xmlns:xacro="http://www.ros.org/wiki/xacro" >
+<robot xmlns:xacro="http://www.ros.org/wiki/xacro" >
   <!--Constant for the robotv1-->
-  <xacro:property name="Pi" value="3.1415926535897931"/>
   <xacro:property name="lenx_hip_2" value="0.04"/>
   <xacro:property name="leny_hip_2" value="0.03"/>
@@ -10,10 +9,10 @@
   <xacro:property name="leny_hip_3" value="0.03"/>
   <xacro:property name="lenz_hip_3" value="0.09"/>
-  <xacro:property name="lenx_upp" value="0.03"/>
-  <xacro:property name="leny_upp" value="0.04"/>
-  <xacro:property name="lenz_upp" value="0.06"/>
-  <xacro:property name="lenx_low" value="0.02"/>
-  <xacro:property name="leny_low" value="0.02"/>
-  <xacro:property name="lenz_low" value="0.14"/>
+  <xacro:property name="lenx_upp_leg" value="0.03"/>
+  <xacro:property name="leny_upp_leg" value="0.04"/>
+  <xacro:property name="lenz_upp_leg" value="0.06"/>
+  <xacro:property name="lenx_low_leg" value="0.02"/>
+  <xacro:property name="leny_low_leg" value="0.02"/>
+  <xacro:property name="lenz_low_leg" value="0.13"/>
   <xacro:property name="lenx_ang_1" value="0.04"/>
   <xacro:property name="leny_ang_1" value="0.03"/>
@@ -24,9 +23,17 @@
   <xacro:property name="lenx_foot" value="0.1"/>
   <xacro:property name="leny_foot" value="0.04"/>
-  <xacro:property name="lenz_foot" value="0.002"/>
-  <xacro:include filename="$(find robotv1_description)/materials/materials.xacro" />
-  <xacro:include filename="$(find robotv1_description)/urdf/robotv1.gazebo" />
+  <xacro:property name="lenz_foot" value="0.02"/>
+  <xacro:property name="base_pos" value="${lenz_hip_3+lenz_upp_leg+lenz_low_leg+lenz_ang_2/2+lenz_foot}"/>
+  <xacro:include filename="$(find robotv1_description)/urdf/leg.gazebo" />
   <xacro:include filename="$(find robotv1_description)/urdf/utilities.xacro"/>
   <xacro:macro name="leg" params="prefix reflect" >
+    <joint name="${prefix}_hip_1_joint" type="revolute" >
+      <parent link="pelvis"/>
+      <child link="${prefix}_hip_2"/>
+      <origin xyz="0 ${leny_pelvis*reflect/2} 0"/>
+      <axis xyz="0 1 0"/>
+      <dynamics damping="0.9"/>
+      <limit effort="2" velocity="1.0" lower="${-pi/2}" upper="${pi/2}" />
+    </joint>
     <link name="${prefix}_hip_2" >
       <visual>
@@ -50,10 +57,10 @@
       <origin xyz= "0 ${leny_hip_2*reflect} 0"/>
       <axis xyz="1 0 0"/>
-      <dynamics damping="0.7"/>
-      <limit effort="20" velocity="1.0" lower="${-Pi/2}" upper="${Pi/2}" />
+      <dynamics damping="0.9"/>
+      <limit effort="2" velocity="1.0" lower="${-pi/2}" upper="${pi/2}" />
     </joint>
     <link name="${prefix}_hip_3" >
       <visual>
-        <origin xyz="0 0 ${-1*lenz_hip_3/2 }" rpy="0 0 0"/>
+        <origin xyz="0 0 ${-lenz_hip_3/2 }" rpy="0 0 0"/>
         <geometry>
           <box size="${lenx_hip_3} ${leny_hip_3} ${lenz_hip_3}"/>
@@ -71,57 +78,57 @@
     <joint name="${prefix}_hip_3_joint" type="revolute" >
       <parent link="${prefix}_hip_3"/>
-      <child link="${prefix}_upp"/>
-      <origin xyz="0 0 ${-1*lenz_hip_3 }"/>
+      <child link="${prefix}_upp_leg"/>
+      <origin xyz="0 0 ${-lenz_hip_3}"/>
       <axis xyz="0 0 1"/>
-      <dynamics damping="0.7"/>
-      <limit effort="20" velocity="1.0" lower="${-Pi/2}" upper="${Pi/2}" />
-    </joint>
-    <link name="${prefix}_upp" >
-      <visual>
-        <origin xyz="0 0 ${-1*lenz_upp/2}" rpy="0 0 0"/>
-        <geometry>
-          <box size="${lenx_upp} ${leny_upp} ${lenz_upp}"/>
+      <dynamics damping="0.9"/>
+      <limit effort="2" velocity="1.0" lower="${-pi/2}" upper="${pi/2}" />
+    </joint>
+    <link name="${prefix}_upp_leg" >
+      <visual>
+        <origin xyz="0 0 ${-lenz_upp_leg/2}" rpy="0 0 0"/>
+        <geometry>
+          <box size="${lenx_upp_leg} ${leny_upp_leg} ${lenz_upp_leg}"/>
         </geometry>
         <material name="black"/>
       </visual>
-     <xacro:box_inertia  lenx="${lenx_upp}" leny="${leny_upp}" lenz="${lenz_upp}" />
-     <collision>
-        <origin xyz="0 0 ${-1*lenz_upp/2}" rpy="0 0 0"/>
-        <geometry>
-          <box size="${lenx_upp} ${leny_upp} ${lenz_upp}"/>
+     <xacro:box_inertia  lenx="${lenx_upp_leg}" leny="${leny_upp_leg}" lenz="${lenz_upp_leg}" />
+     <collision>
+        <origin xyz="0 0 ${-lenz_upp_leg/2}" rpy="0 0 0"/>
+        <geometry>
+          <box size="${lenx_upp_leg} ${leny_upp_leg} ${lenz_upp_leg}"/>
         </geometry>
      </collision>
     </link>
     <joint name="${prefix}_knee_joint" type="revolute" >
-      <parent link="${prefix}_upp"/>
-      <child link="${prefix}_low"/>
-      <origin xyz="0 0 ${-lenz_upp}"/>
+      <parent link="${prefix}_upp_leg"/>
+      <child link="${prefix}_low_leg"/>
+      <origin xyz="0 0 ${-lenz_upp_leg}"/>
       <axis xyz="0 1 0"/>
-      <dynamics damping="0.7"/>
-      <limit effort="20" velocity="1.0" lower="0" upper="${7*Pi/8}" />
-    </joint>
-    <link name="${prefix}_low" >
-      <visual>
-        <origin xyz="0 0 ${-lenz_low/2}" rpy="0 0 0"/>
-        <geometry>
-         <box size="${lenx_low} ${leny_low} ${lenz_low}"/>
+      <dynamics damping="0.9"/>
+      <limit effort="2" velocity="1.0" lower="0" upper="${7*pi/8}" />
+    </joint>
+    <link name="${prefix}_low_leg" >
+      <visual>
+        <origin xyz="0 0 ${-lenz_low_leg/2}" rpy="0 0 0"/>
+        <geometry>
+         <box size="${lenx_low_leg} ${leny_low_leg} ${lenz_low_leg}"/>
         </geometry>
         <material name="orange"/>
       </visual>
-     <xacro:box_inertia  lenx="${lenx_low}" leny="${leny_low}" lenz="${lenz_low}" />
-     <collision>
-       <origin xyz="0 0 ${-lenz_low/2}" rpy="0 0 0"/>
+     <xacro:box_inertia  lenx="${lenx_low_leg}" leny="${leny_low_leg}" lenz="${lenz_low_leg}" />
+     <collision>
+       <origin xyz="0 0 ${-lenz_low_leg/2}" rpy="0 0 0"/>
        <geometry>
-         <box size="${lenx_low} ${leny_low} ${lenz_low}"/>
+         <box size="${lenx_low_leg} ${leny_low_leg} ${lenz_low_leg}"/>
        </geometry>
      </collision>
     </link>
     <joint name="${prefix}_ang_1_joint" type="revolute" >
-      <parent link="${prefix}_low"/>
+      <parent link="${prefix}_low_leg"/>
       <child link="${prefix}_ang_1"/>
-      <origin xyz="0 0 ${-lenz_low+lenz_ang_1/2}" rpy="0 0 0"/>
+      <origin xyz="0 0 ${-lenz_low_leg+lenz_ang_1/2}" rpy="0 0 0"/>
       <axis xyz="1 0 0"/>
-      <dynamics damping="0.7"/>
-      <limit effort="20" velocity="1.0" lower="${-Pi/4}" upper="${Pi/4}" />
+      <dynamics damping="0.9"/>
+      <limit effort="2" velocity="1.0" lower="${-pi/4}" upper="${pi/4}" />
     </joint>
     <link name="${prefix}_ang_1" >
@@ -146,6 +153,6 @@
        <origin xyz="${-lenx_ang_1/2} 0 0"/>
        <axis xyz="0 1 0"/>
-       <dynamics damping="0.7"/>
-       <limit effort="20" velocity="1.0" lower="${-Pi/4}" upper="${Pi/4}" />
+       <dynamics damping="0.9"/>
+       <limit effort="2" velocity="1.0" lower="${-pi/4}" upper="${pi/4}" />
      </joint>
      <link name="${prefix}_ang_2" >
@@ -186,4 +193,14 @@
      </collision>
     </link>
+    <transmission name="${prefix}_hip_1_tran">
+      <type>transmission_interface/SimpleTransmission</type>
+      <joint name="${prefix}_hip_1_joint">
+        <hardwareInterface>hardware_interface/EffortJointInterface</hardwareInterface>
+      </joint>
+      <actuator name="${prefix}_hip_1_motor">
+        <hardwareInterface>hardware_interface/EffortJointInterface</hardwareInterface>
+        <mechanicalReduction>1</mechanicalReduction>
+      </actuator>
+    </transmission>
     <transmission name="${prefix}_hip_2_tran">
       <type>transmission_interface/SimpleTransmission</type>
@@ -236,22 +253,5 @@
       </actuator>
     </transmission>
-    <joint name="${prefix}_hip_1_joint" type="revolute" >
-      <parent link="pelvis"/>
-      <child link="${prefix}_hip_2"/>
-      <origin xyz="0 ${leny_pelvis*reflect/2} 0"/>
-      <axis xyz="0 1 0"/>
-      <dynamics damping="0.7"/>
-      <limit effort="20" velocity="1.0" lower="${-Pi/2}" upper="${Pi/2}" />
-    </joint>
-    <transmission name="${prefix}_hip_1_tran">
-      <type>transmission_interface/SimpleTransmission</type>
-      <joint name="${prefix}_hip_1_joint">
-        <hardwareInterface>hardware_interface/EffortJointInterface</hardwareInterface>
-      </joint>
-      <actuator name="${prefix}_hip_1_motor">
-        <hardwareInterface>hardware_interface/EffortJointInterface</hardwareInterface>
-        <mechanicalReduction>1</mechanicalReduction>
-      </actuator>
-    </transmission>
+   <xacro:leg_gazebo_reference prefix="${prefix}"/>
  </xacro:macro>
 </robot>
