Commit message: updated robotv1 model

File: robotv1_description/urdf/robotv1.xacro (robot description, xacro)
@@ -1,28 +1,18 @@
 <?xml version="1.0"?>
-<!-- Revolute-Revolute Manipulator -->
-<robot name="robotv1" xmlns:xacro="http://www.ros.org/wiki/xacro" >
-  <xacro:include filename="$(find robotv1_description)/urdf/lower_body.xacro"/>
-  <xacro:include filename="$(find robotv1_description)/urdf/upper_body.xacro"/>
-  <link name="world">
-    <inertial>
-      <origin xyz="0 0 1" rpy="0 0 0"/>
-      <mass value="1"/>
-      <inertia
-        ixx="1.0" ixy="0.0" ixz="0.0"
-        iyy="1.0" iyz="0.0"
-        izz="1.0"/>
-    </inertial>
-  </link>
-  <joint name="fixed" type="fixed">
-    <parent link="world"/>
-    <child link="pelvis"/>
-    <origin xyz="0 0 1"/>
-  </joint>
-  <joint name="pelvis_torso_joint" type="fixed">
-    <parent link="pelvis"/>
-    <child link="torso"/>
-    <origin xyz="0 0 ${lenz_pelvis/2}" rpy="0 0 0"/>
-    <axis xyz="0 1 0"/>
-    <limit lower="0" upper="${2*pi}" effort="${elbowEff}" velocity="${elbowVel}"/>
-  </joint>
+<robot name="robotv1" xmlns:xacro="http://www.ros.org/wiki/xacro">
+<xacro:include filename="$(find robotv1_description)/urdf/leg.xacro"/>
+<xacro:include filename="$(find robotv1_description)/urdf/arm.xacro"/>
+<xacro:include filename="$(find robotv1_description)/urdf/torso.xacro"/>
+<xacro:include filename="$(find robotv1_description)/materials/materials.xacro" />
+<!-- only gazebo plug-in -->
+<xacro:include filename="$(find robotv1_description)/urdf/robotv1.gazebo"/>
+<link name="dummy"/>
+<joint name="dummy_to_pelvis" type="fixed">
+  <origin xyz="0 0 ${base_pos}" rpy="0 0 0"/>
+  <parent link="dummy" />
+  <child link="pelvis" />
+</joint>
+<xacro:leg prefix="leftleg" reflect="1"/>
+<xacro:leg prefix="rightleg" reflect="-1"/>
+<xacro:arm prefix="leftarm" />
 </robot>

Commit message: reworked & simplified the simulation model so there are no more collsiions initially (still some depending on joint angles) and the center of mass for each part is correct

File: robotv1_description/urdf/arm.xacro (robot description, xacro)
@@ -4,162 +4,137 @@
   <xacro:include filename="$(find robotv1_description)/urdf/gripper.xacro"/>
   <xacro:include filename="$(find robotv1_description)/urdf/arm.gazebo"/>
-  <xacro:property name="lenx_sho" value="0.06"/>
-  <xacro:property name="leny_sho" value="0.03"/>
-  <xacro:property name="lenz_sho" value="0.04"/>
-  <xacro:property name="lenx_upp_arm" value="0.02"/>
-  <xacro:property name="leny_upp_arm" value="0.06"/>
-  <xacro:property name="lenz_upp_arm" value="0.12"/>
-  <xacro:property name="lenx_low_arm" value="0.02"/>
-  <xacro:property name="leny_low_arm" value="0.04"/>
-  <xacro:property name="lenz_low_arm" value="0.07"/>
-  <xacro:property name="lenx_wri_1" value="0.04"/>
-  <xacro:property name="leny_wri_1" value="0.06"/>
-  <xacro:property name="lenz_wri_1" value="0.03"/>
+  <xacro:property name="lenXUpperArm" value="0.02"/>
+  <xacro:property name="lenYUpperArm" value="0.06"/>
+  <xacro:property name="lenZUpperArm" value="0.12"/>
+  <xacro:property name="lenXLowerArm" value="0.02"/>
+  <xacro:property name="lenYLowerArm" value="0.04"/>
+  <xacro:property name="lenZLowerArm" value="0.07"/>
+  <xacro:property name="lenXWrist" value="0.04"/>
+  <xacro:property name="lenYWrist" value="0.06"/>
+  <xacro:property name="lenZWrist" value="0.03"/>
  <xacro:macro name="arm" params="prefix" >
-    <joint name="${prefix}_shoulder_1_joint" type="revolute" >
-      <parent link="pelvis"/>
-      <child link="${prefix}_sho"/>
-      <origin xyz="0 0 ${lenz_pelvis/2}"/>
-      <axis xyz="0 0 1"/>
-      <dynamics damping="0.7"/>
+    <joint name="${prefix}ShoulderJoint" type="revolute" >
+      <parent link="torso"/>
+      <child link="${prefix}UpperArm"/>
+      <origin xyz="0 0 ${lenZTorso + jointOffset}"/>
+      <axis xyz="0 1 0"/>
+      <dynamics damping="0"/>
       <limit effort="0.2" velocity="1.0" lower="${-pi/2}" upper="${pi/2}" />
     </joint>
-    <link name="${prefix}_sho" >
-      <visual>
-        <origin xyz="0 0 ${lenz_sho/2}" rpy="0 0 0"/>
-        <geometry>
-          <box size="${lenx_sho} ${leny_sho} ${lenz_sho}"/>
-        </geometry>
-        <material name="black"/>
-      </visual>
-      <xacro:box_inertia  lenx="${lenx_sho}" leny="${leny_sho}" lenz="${lenz_sho}" />
-      <collision>
-        <origin xyz="0 0 ${lenz_sho/2}" rpy="0 0 0"/>
-        <geometry>
-          <box size="${lenx_sho} ${leny_sho} ${lenz_sho}"/>
-        </geometry>
-     </collision>
-   </link>
-   <joint name="${prefix}_shoulder_2_joint" type="revolute" >
-     <parent link="${prefix}_sho"/>
-     <child link="${prefix}_upp_arm"/>
-     <origin xyz="0 0 ${lenz_sho/2}"/>
-     <axis xyz="0 1 0"/>
-     <dynamics damping="0.7"/>
-     <limit effort="0.2" velocity="1.0" lower="${-pi/2}" upper="${pi/2}" />
-   </joint>
-   <link name="${prefix}_upp_arm" >
+   <link name="${prefix}UpperArm" >
      <visual>
-       <origin xyz="0 0 ${lenz_upp_arm/2}" rpy="0 0 0"/>
+       <origin xyz="0 0 ${lenZUpperArm/2.0}" rpy="0 0 0"/>
        <geometry>
-         <box size="${lenx_upp_arm} ${leny_upp_arm} ${lenz_upp_arm}"/>
+         <box size="${lenXUpperArm} ${lenYUpperArm} ${lenZUpperArm}"/>
        </geometry>
        <material name="orange"/>
      </visual>
-     <xacro:box_inertia  lenx="${lenx_upp_arm}" leny="${leny_upp_arm}" lenz="${lenz_upp_arm}" />
+     <inertial>
+      <origin xyz="0 0 ${lenZUpperArm/2.0}"/>
+       <xacro:box_inertia  lenx="${lenXUpperArm}" leny="${lenYUpperArm}" lenz="${lenZUpperArm}" />
+     </inertial>
      <collision>
-       <origin xyz="0 0 ${lenz_upp_arm/2}" rpy="0 0 0"/>
+       <origin xyz="0 0 ${lenZUpperArm/2.0}" rpy="0 0 0"/>
        <geometry>
-         <box size="${lenx_upp_arm} ${leny_upp_arm} ${lenz_upp_arm}"/>
+         <box size="${lenXUpperArm} ${lenYUpperArm} ${lenZUpperArm}"/>
        </geometry>
     </collision>
   </link>
-  <joint name="${prefix}_elbow_joint" type="revolute" >
-    <parent link="${prefix}_upp_arm"/>
-    <child link="${prefix}_low_arm"/>
-    <origin xyz="0 0 ${lenz_upp_arm}"/>
+  <joint name="${prefix}ElbowJoint" type="revolute" >
+    <parent link="${prefix}UpperArm"/>
+    <child link="${prefix}LowerArm"/>
+    <origin xyz="0 0 ${lenZUpperArm + jointOffset}"/>
     <axis xyz="0 1 0"/>
-    <dynamics damping="0.7"/>
+    <dynamics damping="0"/>
     <limit effort="0.2" velocity="1.0" lower="0" upper="${pi}" />
   </joint>
-  <link name="${prefix}_low_arm" >
+  <link name="${prefix}LowerArm">
     <visual>
-      <origin xyz="0 0 ${lenz_low_arm/2}" rpy="0 0 0"/>
+      <origin xyz="0 0 ${lenZLowerArm/2}" rpy="0 0 0"/>
       <geometry>
-        <box size="${lenx_low_arm} ${leny_low_arm} ${lenz_low_arm}"/>
+        <box size="${lenXLowerArm} ${lenYLowerArm} ${lenZLowerArm}"/>
       </geometry>
       <material name="black"/>
     </visual>
-    <xacro:box_inertia  lenx="${lenx_low_arm}" leny="${leny_low_arm}" lenz="${lenz_low_arm}" />
+    <inertial>
+      <origin xyz="0 0 ${lenZLowerArm/2.0}"/>
+      <xacro:box_inertia  lenx="${lenXLowerArm}" leny="${lenYLowerArm}" lenz="${lenZLowerArm}" />
+    </inertial>
     <collision>
-      <origin xyz="0 0 ${lenz_low_arm/2}" rpy="0 0 0"/>
+      <origin xyz="0 0 ${lenZLowerArm/2.0}" rpy="0 0 0"/>
       <geometry>
-        <box size="${lenx_low_arm} ${leny_low_arm} ${lenz_low_arm}"/>
+        <box size="${lenXLowerArm} ${lenYLowerArm} ${lenZLowerArm}"/>
       </geometry>
     </collision>
   </link>
-  <joint name="${prefix}_wrist_1_joint" type="revolute" >
-    <parent link="${prefix}_low_arm"/>
-    <child link="${prefix}_wri_1"/>
-    <origin xyz="0 0 ${lenz_low_arm}"/>
+  <joint name="${prefix}WristJoint" type="revolute" >
+    <parent link="${prefix}LowerArm"/>
+    <child link="${prefix}Wrist"/>
+    <origin xyz="0 0 ${lenZLowerArm + jointOffset}"/>
     <axis xyz="0 1 0"/>
-    <dynamics damping="0.7"/>
+    <dynamics damping="0"/>
     <limit effort="0.2" velocity="1.0" lower="${-pi/2}" upper="${pi/2}" />
   </joint>
-  <link name="${prefix}_wri_1" >
+  <link name="${prefix}Wrist" >
     <visual>
-      <origin xyz="0 0 ${lenz_wri_1/2}" rpy="0 0 0"/>
+      <origin xyz="0 0 ${lenZWrist/2}" rpy="0 0 0"/>
       <geometry>
-        <box size="${lenx_wri_1} ${leny_wri_1} ${lenz_wri_1}"/>
+        <box size="${lenXWrist} ${lenYWrist} ${lenZWrist}"/>
       </geometry>
       <material name="orange"/>
     </visual>
-    <xacro:box_inertia  lenx="${lenx_wri_1}" leny="${leny_wri_1}" lenz="${lenz_wri_1}" />
+    <inertial>
+      <origin xyz="0 0 ${lenZWrist/2.0}"/>
+      <xacro:box_inertia  lenx="${lenXWrist}" leny="${lenYWrist}" lenz="${lenZWrist}" />
+    </inertial>
     <collision>
-      <origin xyz="0 0 ${lenz_wri_1/2}" rpy="0 0 0"/>
+      <origin xyz="0 0 ${lenZWrist/2}" rpy="0 0 0"/>
       <geometry>
-        <box size="${lenx_wri_1} ${leny_wri_1} ${lenz_wri_1}"/>
+        <box size="${lenXWrist} ${lenYWrist} ${lenZWrist}"/>
       </geometry>
     </collision>
   </link>
-  <joint name="${prefix}_wrist_2_joint" type="revolute" >
-    <parent link="${prefix}_wri_1"/>
+  <!--
+  <joint name="${prefix}_wrist_2_joint" type="fixed" >
+    <parent link="${prefix}Wrist"/>
     <child link="${prefix}_gripper"/>
-    <origin xyz="0 0 ${lenz_wri_1}"/>
-    <axis xyz="0 0 1"/>
-    <dynamics damping="0.7"/>
+    <origin xyz="0 0 ${lenZWrist}"/>
+    <axis xyz="0 1 0"/>
+    <dynamics damping="0"/>
     <limit effort="0.2" velocity="1.0" lower="${-pi/2}" upper="${pi/2}" />
   </joint>
   <xacro:gripper prefix="${prefix}"/>
-  <transmission name="${prefix}_shoulder_1_joint_tran">
+  -->
+  <transmission name="${prefix}ShoulderTransmission">
     <type> transmission_interface/SimpleTransmission</type>
-    <joint name="${prefix}_shoulder_1_joint">
+    <joint name="${prefix}ShoulderJoint">
       <hardwareInterface>hardware_interface/EffortJointInterface</hardwareInterface>
     </joint>
-    <actuator name="${prefix}_shoulder_1_joint_motor">
+    <actuator name="${prefix}ShoulderMotor">
       <hardwareInterface>hardware_interface/EffortJointInterface</hardwareInterface>
       <mechanicalReduction>1</mechanicalReduction>
     </actuator>
   </transmission>
-  <transmission name="${prefix}_shoulder_2_joint_tran">
+  <transmission name="${prefix}ElbowJointTransmission">
     <type> transmission_interface/SimpleTransmission</type>
-    <joint name="${prefix}_shoulder_2_joint">
+    <joint name="${prefix}ElbowJoint">
       <hardwareInterface>hardware_interface/EffortJointInterface</hardwareInterface>
     </joint>
-    <actuator name="${prefix}_shoulder_2_joint_motor">
+    <actuator name="${prefix}ElbowJointMotor">
       <hardwareInterface>hardware_interface/EffortJointInterface</hardwareInterface>
       <mechanicalReduction>1</mechanicalReduction>
     </actuator>
   </transmission>
-  <transmission name="${prefix}_elbow_joint_tran">
+  <transmission name="${prefix}WristJointTran">
     <type> transmission_interface/SimpleTransmission</type>
-    <joint name="${prefix}_elbow_joint">
+    <joint name="${prefix}WristJoint">
       <hardwareInterface>hardware_interface/EffortJointInterface</hardwareInterface>
     </joint>
-    <actuator name="${prefix}_elbow_joint_motor">
+    <actuator name="${prefix}WristJointMotor">
       <hardwareInterface>hardware_interface/EffortJointInterface</hardwareInterface>
       <mechanicalReduction>1</mechanicalReduction>
     </actuator>
   </transmission>
-  <transmission name="${prefix}_wrist_1_joint_tran">
-    <type> transmission_interface/SimpleTransmission</type>
-    <joint name="${prefix}_wrist_1_joint">
-      <hardwareInterface>hardware_interface/EffortJointInterface</hardwareInterface>
-    </joint>
-    <actuator name="${prefix}_wrist_1_joint_motor">
-      <hardwareInterface>hardware_interface/EffortJointInterface</hardwareInterface>
-      <mechanicalReduction>1</mechanicalReduction>
-    </actuator>
-  </transmission>
+  <!--
   <transmission name="${prefix}_wrist_2_joint_tran">
     <type> transmission_interface/SimpleTransmission</type>
@@ -172,4 +147,5 @@
     </actuator>
   </transmission>
+  -->
   <xacro:arm_gazebo_reference prefix="${prefix}"/>
 </xacro:macro>
