Commit message: reworked & simplified the simulation model so there are no more collsiions initially (still some depending on joint angles) and the center of mass for each part is correct

File: robotv1_description/urdf/leg.xacro (robot description, xacro)
@@ -3,250 +3,123 @@
 <robot xmlns:xacro="http://www.ros.org/wiki/xacro" >
   <!--Constant for the robotv1-->
-  <xacro:property name="lenx_hip_2" value="0.04"/>
-  <xacro:property name="leny_hip_2" value="0.03"/>
-  <xacro:property name="lenz_hip_2" value="0.06"/>
-  <xacro:property name="lenx_hip_3" value="0.07"/>
-  <xacro:property name="leny_hip_3" value="0.03"/>
-  <xacro:property name="lenz_hip_3" value="0.09"/>
-  <xacro:property name="lenx_upp_leg" value="0.03"/>
-  <xacro:property name="leny_upp_leg" value="0.04"/>
-  <xacro:property name="lenz_upp_leg" value="0.06"/>
-  <xacro:property name="lenx_low_leg" value="0.02"/>
-  <xacro:property name="leny_low_leg" value="0.02"/>
-  <xacro:property name="lenz_low_leg" value="0.13"/>
-  <xacro:property name="lenx_ang_1" value="0.04"/>
-  <xacro:property name="leny_ang_1" value="0.03"/>
-  <xacro:property name="lenz_ang_1" value="0.06"/>
-  <xacro:property name="lenx_ang_2" value="0.03"/>
-  <xacro:property name="leny_ang_2" value="0.04"/>
-  <xacro:property name="lenz_ang_2" value="0.06"/>
-  <xacro:property name="lenx_foot" value="0.1"/>
-  <xacro:property name="leny_foot" value="0.04"/>
-  <xacro:property name="lenz_foot" value="0.02"/>
-  <xacro:property name="base_pos" value="${lenz_hip_3+lenz_upp_leg+lenz_low_leg+lenz_ang_2/2+lenz_foot}"/>
   <xacro:include filename="$(find robotv1_description)/urdf/leg.gazebo" />
-  <xacro:include filename="$(find robotv1_description)/urdf/utilities.xacro"/>
+  <xacro:property name="lenXUpperLeg" value="0.06"/>
+  <xacro:property name="lenYUpperLeg" value="0.06"/>
+  <xacro:property name="lenZUpperLeg" value="0.15"/>
+  <xacro:property name="lenXLowerLeg" value="0.06"/>
+  <xacro:property name="lenYLowerLeg" value="0.06"/>
+  <xacro:property name="lenZLowerLeg" value="0.10"/>
+  <xacro:property name="lenXFoot" value="0.1"/>
+  <xacro:property name="lenYFoot" value="0.04"/>
+  <xacro:property name="lenZFoot" value="0.02"/>
+  <xacro:property name="basePosition" value="${lenZUpperLeg+lenZLowerLeg+lenZLowerLeg+lenZFoot}"/>
   <xacro:macro name="leg" params="prefix reflect" >
-    <joint name="${prefix}_hip_1_joint" type="revolute" >
+    <joint name="${prefix}HipJoint" type="revolute" >
       <parent link="pelvis"/>
-      <child link="${prefix}_hip_2"/>
-      <origin xyz="0 ${leny_pelvis*reflect/2} 0"/>
+      <child link="${prefix}UpperLeg"/>
+      <origin xyz="0 ${reflect*(lenYUpperLeg/2.0 + lenYPelvis/2.0 + jointOffset)} 0"/>
       <axis xyz="0 1 0"/>
-      <dynamics damping="0.9"/>
+      <dynamics damping="0"/>
       <limit effort="2" velocity="1.0" lower="${-pi/2}" upper="${pi/2}" />
     </joint>
-    <link name="${prefix}_hip_2" >
+    <link name="${prefix}UpperLeg" >
       <visual>
-        <origin xyz="0 ${leny_hip_2*reflect/2} 0" rpy="0 0 0"/>
+        <origin xyz="0 0 ${-1*lenZUpperLeg/2.0}" rpy="0 0 0"/>
         <geometry>
-          <box size="${lenx_hip_2} ${leny_hip_2} ${lenz_hip_2}"/>
+          <box size="${lenXUpperLeg} ${lenYUpperLeg} ${lenZUpperLeg}"/>
         </geometry>
         <material name="black"/>
       </visual>
-      <xacro:box_inertia  lenx="${lenx_hip_2}" leny="${leny_hip_2}" lenz="${lenz_hip_2}" />
+      <inertial>
+        <origin xyz="0 0 ${-1*lenZUpperLeg/2.0}"/>
+        <xacro:box_inertia  lenx="${lenXUpperLeg}" leny="${lenYUpperLeg}" lenz="${lenZUpperLeg}" />
+      </inertial>
       <collision>
-        <origin xyz="0 ${leny_hip_2*reflect/2} 0" rpy="0 0 0"/>
+        <origin xyz="0 0 ${-1*lenZUpperLeg/2.0}" rpy="0 0 0"/>
         <geometry>
-          <box size="${lenx_hip_2} ${leny_hip_2} ${lenz_hip_2}"/>
+          <box size="${lenXUpperLeg} ${lenYUpperLeg} ${lenZUpperLeg}"/>
         </geometry>
      </collision>
    </link>
-   <joint name="${prefix}_hip_2_joint" type="revolute" >
-      <parent link="${prefix}_hip_2"/>
-      <child link="${prefix}_hip_3"/>
-      <origin xyz= "0 ${leny_hip_2*reflect} 0"/>
-      <axis xyz="1 0 0"/>
-      <dynamics damping="0.9"/>
-      <limit effort="2" velocity="1.0" lower="${-pi/2}" upper="${pi/2}" />
+    <joint name="${prefix}KneeJoint" type="revolute" >
+      <parent link="${prefix}UpperLeg"/>
+      <child link="${prefix}LowerLeg"/>
+      <origin xyz="0 0 ${-lenZUpperLeg - jointOffset}" rpy = "0 0 0"/>
+      <axis xyz="0 1 0"/>
+      <dynamics damping="0"/>
+      <limit effort="2" velocity="1.0" lower="0" upper="${7*pi/8}" />
     </joint>
-    <link name="${prefix}_hip_3" >
+    <link name="${prefix}LowerLeg" >
       <visual>
-        <origin xyz="0 0 ${-lenz_hip_3/2 }" rpy="0 0 0"/>
+        <origin xyz="0 0 ${-lenZLowerLeg/2.0}" rpy="0 0 0"/>
         <geometry>
-          <box size="${lenx_hip_3} ${leny_hip_3} ${lenz_hip_3}"/>
+         <box size="${lenXLowerLeg} ${lenYLowerLeg} ${lenZLowerLeg}"/>
         </geometry>
         <material name="orange"/>
       </visual>
-     <xacro:box_inertia  lenx="${lenx_hip_3}" leny="${leny_hip_3}" lenz="${lenz_hip_3}" />
+    <inertial>
+      <origin xyz="0 0 ${-1*lenZLowerLeg/2.0}"/>
+      <xacro:box_inertia  lenx="${lenXLowerLeg}" leny="${lenYLowerLeg}" lenz="${lenZLowerLeg}" />
+    </inertial>
      <collision>
-        <origin xyz="0 0 ${-1*lenz_hip_3/2 }" rpy="0 0 0"/>
-        <geometry>
-          <box size="${lenx_hip_3} ${leny_hip_3} ${lenz_hip_3}"/>
-        </geometry>
+       <origin xyz="0 0 ${-lenZLowerLeg/2.0}" rpy="0 0 0"/>
+       <geometry>
+         <box size="${lenXLowerLeg} ${lenYLowerLeg} ${lenZLowerLeg}"/>
+       </geometry>
      </collision>
     </link>
-    <joint name="${prefix}_hip_3_joint" type="revolute" >
-      <parent link="${prefix}_hip_3"/>
-      <child link="${prefix}_upp_leg"/>
-      <origin xyz="0 0 ${-lenz_hip_3}"/>
-      <axis xyz="0 0 1"/>
-      <dynamics damping="0.9"/>
-      <limit effort="2" velocity="1.0" lower="${-pi/2}" upper="${pi/2}" />
+    <joint name="${prefix}AnkleJoint" type="revolute" >
+      <parent link="${prefix}LowerLeg"/>
+      <child link="${prefix}Foot"/>
+      <origin xyz="0 0 ${-lenZLowerLeg - jointOffset}" rpy="0 0 0"/>
+      <axis xyz="0 1 0"/>
+      <dynamics damping="0"/>
+      <limit effort="2" velocity="1.0" lower="${-pi/4}" upper="${pi/4}" />
     </joint>
-    <link name="${prefix}_upp_leg" >
+    <link name="${prefix}Foot" >
       <visual>
-        <origin xyz="0 0 ${-lenz_upp_leg/2}" rpy="0 0 0"/>
+        <origin xyz="${lenXFoot/2} 0 ${-lenZFoot/2}" rpy="0 0 0"/>
         <geometry>
-          <box size="${lenx_upp_leg} ${leny_upp_leg} ${lenz_upp_leg}"/>
-        </geometry>
-        <material name="black"/>
-      </visual>
-     <xacro:box_inertia  lenx="${lenx_upp_leg}" leny="${leny_upp_leg}" lenz="${lenz_upp_leg}" />
-     <collision>
-        <origin xyz="0 0 ${-lenz_upp_leg/2}" rpy="0 0 0"/>
-        <geometry>
-          <box size="${lenx_upp_leg} ${leny_upp_leg} ${lenz_upp_leg}"/>
-        </geometry>
-     </collision>
-    </link>
-    <joint name="${prefix}_knee_joint" type="revolute" >
-      <parent link="${prefix}_upp_leg"/>
-      <child link="${prefix}_low_leg"/>
-      <origin xyz="0 0 ${-lenz_upp_leg}"/>
-      <axis xyz="0 1 0"/>
-      <dynamics damping="0.9"/>
-      <limit effort="2" velocity="1.0" lower="0" upper="${7*pi/8}" />
-    </joint>
-    <link name="${prefix}_low_leg" >
-      <visual>
-        <origin xyz="0 0 ${-lenz_low_leg/2}" rpy="0 0 0"/>
-        <geometry>
-         <box size="${lenx_low_leg} ${leny_low_leg} ${lenz_low_leg}"/>
+          <box size="${lenXFoot} ${lenYFoot} ${lenZFoot}"/>
         </geometry>
         <material name="orange"/>
       </visual>
-     <xacro:box_inertia  lenx="${lenx_low_leg}" leny="${leny_low_leg}" lenz="${lenz_low_leg}" />
+     <inertial>
+       <origin xyz="${lenXFoot/2.0} 0 ${-lenZFoot/2.0}"/>
+       <xacro:box_inertia  lenx="${lenXFoot}" leny="${lenYFoot}" lenz="${lenZFoot}" />
+     </inertial>
      <collision>
-       <origin xyz="0 0 ${-lenz_low_leg/2}" rpy="0 0 0"/>
+       <origin xyz="${lenXFoot/2} 0 ${-lenZFoot/2}" rpy="0 0 0"/>
        <geometry>
-         <box size="${lenx_low_leg} ${leny_low_leg} ${lenz_low_leg}"/>
+          <box size="${lenXFoot} ${lenYFoot} ${lenZFoot}"/>
        </geometry>
      </collision>
     </link>
-    <joint name="${prefix}_ang_1_joint" type="revolute" >
-      <parent link="${prefix}_low_leg"/>
-      <child link="${prefix}_ang_1"/>
-      <origin xyz="0 0 ${-lenz_low_leg+lenz_ang_1/2}" rpy="0 0 0"/>
-      <axis xyz="1 0 0"/>
-      <dynamics damping="0.9"/>
-      <limit effort="2" velocity="1.0" lower="${-pi/4}" upper="${pi/4}" />
-    </joint>
-    <link name="${prefix}_ang_1" >
-      <visual>
-      <origin xyz="0 0 0" rpy="0 0 0"/>
-        <geometry>
-          <box size="${lenx_ang_1} ${leny_ang_1} ${lenz_ang_1}"/>
-        </geometry>
-        <material name="black"/>
-      </visual>
-     <xacro:box_inertia  lenx="${lenx_ang_1}" leny="${leny_ang_1}" lenz="${lenz_ang_1}" />
-     <collision>
-       <origin xyz="0 0 0" rpy="0 0 0"/>
-       <geometry>
-         <box size="${lenx_ang_1} ${leny_ang_1} ${lenz_ang_1}"/>
-       </geometry>
-      </collision>
-     </link>
-     <joint name="${prefix}_ang_2_joint" type="revolute" >
-       <parent link="${prefix}_ang_1"/>
-       <child link="${prefix}_ang_2"/>
-       <origin xyz="${-lenx_ang_1/2} 0 0"/>
-       <axis xyz="0 1 0"/>
-       <dynamics damping="0.9"/>
-       <limit effort="2" velocity="1.0" lower="${-pi/4}" upper="${pi/4}" />
-     </joint>
-     <link name="${prefix}_ang_2" >
-       <visual>
-       <origin xyz="0 0 ${-lenz_ang_2/2}" rpy="0 0 0"/>
-         <geometry>
-           <box size="${lenx_ang_2} ${leny_ang_2} ${lenz_ang_2}"/>
-         </geometry>
-         <material name="orange"/>
-       </visual>
-     <xacro:box_inertia  lenx="${lenx_ang_2}" leny="${leny_ang_2}" lenz="${lenz_ang_2}" />
-      <collision>
-       <origin xyz="${-lenx_ang_1} 0 ${-lenz_ang_2/2}" rpy="0 0 0"/>
-        <geometry>
-          <box size="${lenx_ang_2} ${leny_ang_2} ${lenz_ang_2}"/>
-        </geometry>
-      </collision>
-    </link>
-    <joint name="${prefix}_foot_joint" type="fixed" >
-      <parent link="${prefix}_ang_2"/>
-      <child link="${prefix}_foot"/>
-      <origin xyz="0 0 ${-lenz_ang_2}"/>
-    </joint>
-    <link name="${prefix}_foot" >
-      <visual>
-        <origin xyz="${lenx_foot/2-lenx_ang_2/2} 0 ${-lenz_foot/2}" rpy="0 0 0"/>
-        <geometry>
-          <box size="${lenx_foot} ${leny_foot} ${lenz_foot}"/>
-        </geometry>
-        <material name="orange"/>
-      </visual>
-     <xacro:box_inertia  lenx="${lenx_foot}" leny="${leny_foot}" lenz="${lenz_foot}" />
-     <collision>
-       <origin xyz="${lenx_foot/2-lenx_ang_2/2} 0 ${-lenz_foot/2}" rpy="0 0 0"/>
-       <geometry>
-          <box size="${lenx_foot} ${leny_foot} ${lenz_foot}"/>
-       </geometry>
-     </collision>
-    </link>
-    <transmission name="${prefix}_hip_1_tran">
+    <transmission name="${prefix}HipTransmission">
       <type>transmission_interface/SimpleTransmission</type>
-      <joint name="${prefix}_hip_1_joint">
+      <joint name="${prefix}HipJoint">
         <hardwareInterface>hardware_interface/EffortJointInterface</hardwareInterface>
       </joint>
-      <actuator name="${prefix}_hip_1_motor">
+      <actuator name="${prefix}HipMotor">
         <hardwareInterface>hardware_interface/EffortJointInterface</hardwareInterface>
         <mechanicalReduction>1</mechanicalReduction>
       </actuator>
     </transmission>
-    <transmission name="${prefix}_hip_2_tran">
+    <transmission name="${prefix}KneeTransmission">
       <type>transmission_interface/SimpleTransmission</type>
-      <joint name="${prefix}_hip_2_joint">
+      <joint name="${prefix}KneeJoint">
         <hardwareInterface>hardware_interface/EffortJointInterface</hardwareInterface>
       </joint>
-      <actuator name="${prefix}_hip_2_motor">
+      <actuator name="${prefix}KneeMotor">
         <hardwareInterface>hardware_interface/EffortJointInterface</hardwareInterface>
         <mechanicalReduction>1</mechanicalReduction>
       </actuator>
     </transmission>
-    <transmission name="${prefix}_hip_3_tran">
+    <transmission name="${prefix}AnkleTransmission">
       <type>transmission_interface/SimpleTransmission</type>
-      <joint name="${prefix}_hip_3_joint">
+      <joint name="${prefix}AnkleJoint">
         <hardwareInterface>hardware_interface/EffortJointInterface</hardwareInterface>
       </joint>
-      <actuator name="${prefix}_hip_3_motor">
-        <hardwareInterface>hardware_interface/EffortJointInterface</hardwareInterface>
-        <mechanicalReduction>1</mechanicalReduction>
-      </actuator>
-    </transmission>
-    <transmission name="${prefix}_knee_tran">
-      <type>transmission_interface/SimpleTransmission</type>
-      <joint name="${prefix}_knee_joint">
-        <hardwareInterface>hardware_interface/EffortJointInterface</hardwareInterface>
-      </joint>
-      <actuator name="${prefix}_knee_motor">
-        <hardwareInterface>hardware_interface/EffortJointInterface</hardwareInterface>
-        <mechanicalReduction>1</mechanicalReduction>
-      </actuator>
-    </transmission>
-    <transmission name="${prefix}_ang_1_tran">
-      <type>transmission_interface/SimpleTransmission</type>
-      <joint name="${prefix}_ang_1_joint">
-        <hardwareInterface>hardware_interface/EffortJointInterface</hardwareInterface>
-      </joint>
-      <actuator name="${prefix}_ang_1_motor">
-        <hardwareInterface>hardware_interface/EffortJointInterface</hardwareInterface>
-        <mechanicalReduction>1</mechanicalReduction>
-      </actuator>
-    </transmission>
-    <transmission name="${prefix}_ang_2_tran">
-      <type>transmission_interface/SimpleTransmission</type>
-      <joint name="${prefix}_ang_2_joint">
-        <hardwareInterface>hardware_interface/EffortJointInterface</hardwareInterface>
-      </joint>
-      <actuator name="${prefix}_ang_2_motor">
+      <actuator name="${prefix}AnkleMotor">
         <hardwareInterface>hardware_interface/EffortJointInterface</hardwareInterface>
         <mechanicalReduction>1</mechanicalReduction>

File: robotv1_description/urdf/lower_body.xacro (robot description, xacro)
@@ -2,24 +2,27 @@
 <robot name="upper_body" xmlns:xacro="http://www.ros.org/wiki/xacro">
   <xacro:include filename="$(find robotv1_description)/urdf/leg.xacro"/>
-  <xacro:property name="lenx_pelvis" value="0.08"/>
-  <xacro:property name="leny_pelvis" value="0.16"/>
-  <xacro:property name="lenz_pelvis" value="0.06"/>
+  <xacro:property name="lenXPelvis" value="0.08"/>
+  <xacro:property name="lenYPelvis" value="0.16"/>
+  <xacro:property name="lenZPelvis" value="0.06"/>
   <link name="pelvis" >
     <visual>
-      <origin xyz="0 0 0 " rpy="0 0 0" />
+      <origin xyz="0 0 0" rpy="0 0 0" />
       <geometry>
-        <box size="${lenx_pelvis} ${leny_pelvis} ${lenz_pelvis}"/>
+        <box size="${lenXPelvis} ${lenYPelvis} ${lenZPelvis}"/>
       </geometry>
       <material name="orange"/>
     </visual>
-    <xacro:box_inertia lenx="${lenx_pelvis}" leny="${leny_pelvis}" lenz="${lenz_pelvis}"/>
+    <inertial>
+      <origin xyz="0 0 0"/>
+      <xacro:box_inertia lenx="${lenXPelvis}" leny="${lenYPelvis}" lenz="${lenZPelvis}"/>
+    </inertial>
     <collision>
-      <origin xyz="0 0 0 " rpy="0 0 0" />
+      <origin xyz="0 0 0" rpy="0 0 0" />
       <geometry>
-        <box size="${lenx_pelvis} ${leny_pelvis} ${lenz_pelvis}"/>
+        <box size="${lenXPelvis} ${lenYPelvis} ${lenZPelvis}"/>
       </geometry>
     </collision>
   </link>
-  <xacro:leg prefix="left_leg" reflect="1" />
-  <xacro:leg prefix="right_leg" reflect="-1" />
+  <xacro:leg prefix="left" reflect="1" />
+  <xacro:leg prefix="right" reflect="-1" />
 </robot>

File: robotv1_description/urdf/robotv1.xacro (robot description, xacro)
@@ -1,18 +1,20 @@
 <?xml version="1.0"?>
 <robot name="robotv1" xmlns:xacro="http://www.ros.org/wiki/xacro">
-<xacro:include filename="$(find robotv1_description)/urdf/leg.xacro"/>
-<xacro:include filename="$(find robotv1_description)/urdf/arm.xacro"/>
-<xacro:include filename="$(find robotv1_description)/urdf/torso.xacro"/>
+<xacro:include filename="$(find robotv1_description)/urdf/utilities.xacro"/>
+<xacro:include filename="$(find robotv1_description)/urdf/lower_body.xacro"/>
+<xacro:include filename="$(find robotv1_description)/urdf/upper_body.xacro"/>
 <xacro:include filename="$(find robotv1_description)/materials/materials.xacro" />
 <!-- only gazebo plug-in -->
 <xacro:include filename="$(find robotv1_description)/urdf/robotv1.gazebo"/>
-<link name="dummy"/>
-<joint name="dummy_to_pelvis" type="fixed">
-  <origin xyz="0 0 ${base_pos}" rpy="0 0 0"/>
-  <parent link="dummy" />
+<link name="world"/>
+<joint name="fixed_world" type="fixed">
+  <origin xyz="0 0 ${basePosition}" rpy="0 0 0"/>
+  <parent link="world" />
   <child link="pelvis" />
 </joint>
-<xacro:leg prefix="leftleg" reflect="1"/>
-<xacro:leg prefix="rightleg" reflect="-1"/>
-<xacro:arm prefix="leftarm" />
+<joint name="pelvisTorsoJoint" type="fixed">
+  <origin xyz="0 0 ${lenZPelvis/2.0 + jointOffset}"/>
+  <parent link="pelvis"/>
+  <child link="torso"/>
+</joint>
 </robot>

File: robotv1_description/urdf/upper_body.xacro (robot description, xacro)
@@ -1,71 +1,27 @@
 <robot name="robotv1" xmlns:xacro="http://www.ros.org/wiki/xacro">
-  <xacro:include filename="$(find robotv1_description)/urdf/robotv1.gazebo"/>
   <xacro:include filename="$(find robotv1_description)/urdf/utilities.xacro"/>
-  <xacro:property name="torsoZ" value=".1"/>
-  <xacro:property name="torsoY" value=".05"/>
-  <xacro:property name="torsoX" value=".05"/>
   <xacro:include filename="$(find robotv1_description)/urdf/arm.xacro"/>
-  <xacro:include filename="$(find robotv1_description)/urdf/gripper.xacro"/>
-  <xacro:robot_v1_arm prefix="left" reflect="1.0"/>
-  <xacro:robot_v1_gripper prefix="left"/>
+  <xacro:property name="lenZTorso" value=".1"/>
+  <xacro:property name="lenYTorso" value=".05"/>
+  <xacro:property name="lenXTorso" value=".05"/>
   <link name="torso">
     <visual>
-      <origin xyz="0 0 ${torsoZ/2}" rpy="0 0 0"/>
+      <origin xyz="0 0 ${lenZTorso/2}" rpy="0 0 0"/>
       <geometry>
-        <box size="${torsoX} ${torsoY} ${torsoZ}"/>
+        <box size="${lenXTorso} ${lenYTorso} ${lenZTorso}"/>
       </geometry>
       <material name="black"/>
     </visual>
     <collision>
-      <origin xyz="0 0 ${torsoZ/2}" rpy="0 0 0"/>
+      <origin xyz="0 0 ${lenZTorso/2}" rpy="0 0 0"/>
       <geometry>
-        <box size="${torsoX} ${torsoY} ${torsoZ}"/>
+        <box size="${lenXTorso} ${lenYTorso} ${lenZTorso}"/>
       </geometry>
     </collision>
-    <xacro:box_inertia lenx="${torsoX}" leny="${torsoY}" lenz="${torsoZ}"/>
+    <inertial>
+      <origin xyz="0 0 ${lenZTorso}"/>
+      <xacro:box_inertia lenx="${lenXTorso}" leny="${lenYTorso}" lenz="${lenZTorso}"/>
+    </inertial>
   </link>
-  <joint name="shoulder" type="revolute">
-    <parent link="torso"/>
-    <child link="left_upper_arm"/>
-    <origin xyz="0 ${0} ${torsoZ}" rpy="0 ${pi*2/3} 0"/>
-    <axis xyz="0 1 0"/>
-    <limit lower="0" upper="${2*pi}" effort="${elbowEff}" velocity="${elbowVel}"/>
-  </joint>
-  <joint name="wrist" type="revolute">
-    <parent link="left_lower_arm"/>
-    <child link="left_gripper"/>
-    <origin xyz="0 0 ${lowerArmLength}" rpy="0 0 0"/>
-    <axis xyz="0 1 0"/>
-    <limit lower="0" upper="${2*pi}" effort="${elbowEff}" velocity="${elbowVel}"/>
-  </joint>
-  <transmission name="shoulder_trans">
-    <type> transmission_interface/SimpleTransmission</type>
-    <joint name="shoulder">
-      <hardwareInterface>hardware_interface/EffortJointInterface</hardwareInterface>
-    </joint>
-    <actuator name="shoulder_motor">
-      <hardwareInterface>hardware_interface/EffortJointInterface</hardwareInterface>
-      <mechanicalReduction>1</mechanicalReduction>
-    </actuator>
-  </transmission>
-  <transmission name="elbow_trans">
-    <type> transmission_interface/SimpleTransmission</type>
-    <joint name="elbow">
-      <hardwareInterface>hardware_interface/EffortJointInterface</hardwareInterface>
-    </joint>
-    <actuator name="elbow_motor">
-      <hardwareInterface>hardware_interface/EffortJointInterface</hardwareInterface>
-      <mechanicalReduction>1</mechanicalReduction>
-    </actuator>
-  </transmission>
-  <transmission name="wrist_trans">
-    <type> transmission_interface/SimpleTransmission</type>
-    <joint name="wrist">
-      <hardwareInterface>hardware_interface/EffortJointInterface</hardwareInterface>
-    </joint>
-    <actuator name="wrist_motor">
-      <hardwareInterface>hardware_interface/EffortJointInterface</hardwareInterface>
-      <mechanicalReduction>1</mechanicalReduction>
-    </actuator>
-  </transmission>
+  <xacro:arm prefix=""/>
 </robot>

File: robotv1_description/urdf/utilities.xacro (robot description, xacro)
@@ -2,13 +2,12 @@
 <robot xmlns:xacro="http://www.ros.org/wiki/xacro">
   <xacro:property name="density" value="2700"/>
+  <xacro:property name="jointOffset" value="0.01"/>
   <xacro:macro name="box_inertia" params="lenx leny lenz">
     <xacro:property name="mass" value="${density * lenx * leny * lenz}"/>
-    <inertial>
-      <mass value="${mass}" />
+      <mass value="${mass}"/>
       <inertia
       ixx="${mass*(lenz*lenz+leny*leny)/12.0}" ixy="0.0" ixz="0.0"
       iyy="${mass*(lenz*lenz+lenx*lenx)/12.0}" iyz="0.0"
       izz="${mass*(lenx*lenx+leny*leny)/12.0}" />
-    </inertial>
   </xacro:macro>
 </robot>
