Commit message: rewrite the model damping=0.03

File: robotv1_description/urdf/leg.xacro (robot description, xacro)
@@ -3,254 +3,308 @@
 <robot xmlns:xacro="http://www.ros.org/wiki/xacro" >
   <!--Constant for the robotv1-->
-  <xacro:property name="lenx_hip_2" value="0.04"/>
-  <xacro:property name="leny_hip_2" value="0.03"/>
-  <xacro:property name="lenz_hip_2" value="0.06"/>
-  <xacro:property name="lenx_hip_3" value="0.07"/>
-  <xacro:property name="leny_hip_3" value="0.03"/>
-  <xacro:property name="lenz_hip_3" value="0.09"/>
-  <xacro:property name="lenx_upp_leg" value="0.03"/>
-  <xacro:property name="leny_upp_leg" value="0.04"/>
-  <xacro:property name="lenz_upp_leg" value="0.06"/>
-  <xacro:property name="lenx_low_leg" value="0.02"/>
-  <xacro:property name="leny_low_leg" value="0.02"/>
-  <xacro:property name="lenz_low_leg" value="0.13"/>
-  <xacro:property name="lenx_ang_1" value="0.04"/>
-  <xacro:property name="leny_ang_1" value="0.03"/>
-  <xacro:property name="lenz_ang_1" value="0.06"/>
-  <xacro:property name="lenx_ang_2" value="0.03"/>
-  <xacro:property name="leny_ang_2" value="0.04"/>
-  <xacro:property name="lenz_ang_2" value="0.06"/>
-  <xacro:property name="lenx_foot" value="0.1"/>
-  <xacro:property name="leny_foot" value="0.04"/>
-  <xacro:property name="lenz_foot" value="0.02"/>
-  <xacro:property name="base_pos" value="${lenz_hip_3+lenz_upp_leg+lenz_low_leg+lenz_ang_2/2+lenz_foot}"/>
+  <xacro:property name="joint_friction" value="0.015"/>
+  <xacro:property name="joint_damping" value="0.03"/>
+  <xacro:property name="joint_effort" value="10.0"/>
+  <xacro:property name="joint_vel" value="3.0"/>
+  <xacro:property name="lx_u0" value="0.04"/>
+  <xacro:property name="ly_u0" value="0.03"/>
+  <xacro:property name="lz_u0" value="0.06"/>
+  <xacro:property name="lx_u1" value="0.06"/>
+  <xacro:property name="ly_u1" value="0.03"/>
+  <xacro:property name="lz_u1" value="0.09"/>
+  <xacro:property name="lx_u2" value="0.03"/>
+  <xacro:property name="ly_u2" value="0.04"/>
+  <xacro:property name="lz_u2" value="0.06"/>
+  <xacro:property name="lx_l0" value="0.015"/>
+  <xacro:property name="ly_l0" value="0.015"/>
+  <xacro:property name="lz_l0" value="0.16"/>
+  <xacro:property name="lx_l1" value="0.04"/>
+  <xacro:property name="ly_l1" value="0.03"/>
+  <xacro:property name="lz_l1" value="0.06"/>
+  <xacro:property name="lx_l2" value="0.03"/>
+  <xacro:property name="ly_l2" value="0.04"/>
+  <xacro:property name="lz_l2" value="0.06"/>
+  <xacro:property name="lx_l3" value="0.1"/>
+  <xacro:property name="ly_l3" value="0.04"/>
+  <xacro:property name="lz_l3" value="0.01"/>
+  <xacro:property name="lx_imu_link" value="0.03"/>
+  <xacro:property name="ly_imu_link" value="0.03"/>
+  <xacro:property name="lz_imu_link" value="0.005"/>
   <xacro:include filename="$(find robotv1_description)/urdf/leg.gazebo" />
   <xacro:include filename="$(find robotv1_description)/urdf/utilities.xacro"/>
   <xacro:macro name="leg" params="prefix reflect" >
-    <joint name="${prefix}_hip_1_joint" type="revolute" >
+    <joint name="${prefix}_H0" type="revolute" >
       <parent link="pelvis"/>
-      <child link="${prefix}_hip_2"/>
-      <origin xyz="0 ${leny_pelvis*reflect/2} 0"/>
+      <child link="${prefix}_u0"/>
+      <origin xyz="0 ${ly_pelvis*reflect/2} 0"/>
       <axis xyz="0 1 0"/>
-      <dynamics damping="0.9"/>
-      <limit effort="2" velocity="1.0" lower="${-pi/2}" upper="${pi/2}" />
-    </joint>
-    <link name="${prefix}_hip_2" >
-      <visual>
-        <origin xyz="0 ${leny_hip_2*reflect/2} 0" rpy="0 0 0"/>
-        <geometry>
-          <box size="${lenx_hip_2} ${leny_hip_2} ${lenz_hip_2}"/>
+      <dynamics damping="${joint_damping}" friction="${joint_friction}"/>
+      <limit effort="${joint_effort}" velocity="${joint_vel}" lower="${-pi/2}" upper="${pi/2}" />
+      <!--
+      <safety_controller k_velocity="10" k_position="15" soft_lower_limit="${-7*pi/8}" soft_upper_limit="${7*pi/8}" />
+       -->
+    </joint>
+    <transmission name="${prefix}_H0_tran">
+      <type>transmission_interface/SimpleTransmission</type>
+      <joint name="${prefix}_H0">
+        <hardwareInterface>hardware_interface/EffortJointInterface</hardwareInterface>
+      </joint>
+      <actuator name="${prefix}_H0_motor">
+        <hardwareInterface>hardware_interface/EffortJointInterface</hardwareInterface>
+        <mechanicalReduction>1</mechanicalReduction>
+      </actuator>
+    </transmission>
+    <link name="${prefix}_u0" >
+      <visual>
+        <origin xyz="0 ${ly_u0*reflect/2} 0" rpy="0 0 0"/>
+        <geometry>
+          <box size="${lx_u0} ${ly_u0} ${lz_u0}"/>
         </geometry>
         <material name="black"/>
       </visual>
-      <xacro:box_inertia  lenx="${lenx_hip_2}" leny="${leny_hip_2}" lenz="${lenz_hip_2}" />
-      <collision>
-        <origin xyz="0 ${leny_hip_2*reflect/2} 0" rpy="0 0 0"/>
-        <geometry>
-          <box size="${lenx_hip_2} ${leny_hip_2} ${lenz_hip_2}"/>
-        </geometry>
-     </collision>
-   </link>
-   <joint name="${prefix}_hip_2_joint" type="revolute" >
-      <parent link="${prefix}_hip_2"/>
-      <child link="${prefix}_hip_3"/>
-      <origin xyz= "0 ${leny_hip_2*reflect} 0"/>
+      <inertial>
+        <origin xyz="0 ${ly_u0*reflect/2} 0" rpy="0 0 0"/>
+        <xacro:box_inertia  lenx="${lx_u0}" leny="${ly_u0}" lenz="${lz_u0}" />
+      </inertial>
+      <collision>
+        <origin xyz="0 ${ly_u0*reflect/2} 0" rpy="0 0 0"/>
+        <geometry>
+          <box size="${lx_u0} ${ly_u0} ${lz_u0}"/>
+        </geometry>
+      </collision>
+    </link>
+    <joint name="${prefix}_H1" type="revolute" >
+       <parent link="${prefix}_u0"/>
+       <child link="${prefix}_u1"/>
+       <origin xyz= "0 ${ly_u0*reflect} 0"/>
+       <axis xyz="1 0 0"/>
+       <dynamics damping="${joint_damping}" friction="${joint_friction}"/>
+       <limit effort="${joint_effort}" velocity="${joint_vel}" lower="${-pi/2}" upper="${pi/2}" />
+    </joint>
+    <transmission name="${prefix}_H1_tran">
+      <type>transmission_interface/SimpleTransmission</type>
+      <joint name="${prefix}_H1">
+        <hardwareInterface>hardware_interface/EffortJointInterface</hardwareInterface>
+      </joint>
+      <actuator name="${prefix}_H1_motor">
+        <hardwareInterface>hardware_interface/EffortJointInterface</hardwareInterface>
+        <mechanicalReduction>1</mechanicalReduction>
+      </actuator>
+    </transmission>
+    <link name="${prefix}_u1" >
+      <visual>
+        <origin xyz="0 0 ${-lz_u1/2 }" rpy="0 0 0"/>
+        <geometry>
+          <box size="${lx_u1} ${ly_u1} ${lz_u1}"/>
+        </geometry>
+        <material name="orange"/>
+      </visual>
+      <inertial>
+        <origin xyz="0 0 ${-lz_u1/2 }" rpy="0 0 0"/>
+        <xacro:box_inertia  lenx="${lx_u1}" leny="${ly_u1}" lenz="${lz_u1}" />
+      </inertial>
+      <collision>
+        <origin xyz="0 0 ${-1*lz_u1/2 }" rpy="0 0 0"/>
+        <geometry>
+          <box size="${lx_u1} ${ly_u1} ${lz_u1}"/>
+        </geometry>
+      </collision>
+    </link>
+    <joint name="${prefix}_H2" type="revolute" >
+      <parent link="${prefix}_u1"/>
+      <child link="${prefix}_u2"/>
+      <origin xyz="0 0 ${-lz_u1}"/>
+      <axis xyz="0 0 1"/>
+      <dynamics damping="${joint_damping}" friction="${joint_friction}"/>
+      <limit effort="${joint_effort}" velocity="${joint_vel}" lower="${-pi/2}" upper="${pi/2}" />
+    </joint>
+    <transmission name="${prefix}_H2_tran">
+      <type>transmission_interface/SimpleTransmission</type>
+      <joint name="${prefix}_H2">
+        <hardwareInterface>hardware_interface/EffortJointInterface</hardwareInterface>
+      </joint>
+      <actuator name="${prefix}_H2_motor">
+        <hardwareInterface>hardware_interface/EffortJointInterface</hardwareInterface>
+        <mechanicalReduction>1</mechanicalReduction>
+      </actuator>
+    </transmission>
+    <link name="${prefix}_u2" >
+      <visual>
+        <origin xyz="0 0 ${-lz_u2/2}" rpy="0 0 0"/>
+        <geometry>
+          <box size="${lx_u2} ${ly_u2} ${lz_u2}"/>
+        </geometry>
+        <material name="black"/>
+      </visual>
+      <inertial>
+        <origin xyz="0 0 ${-lz_u2/2}" rpy="0 0 0"/>
+        <xacro:box_inertia  lenx="${lx_u2}" leny="${ly_u2}" lenz="${lz_u2}" />
+      </inertial>
+      <collision>
+        <origin xyz="0 0 ${-lz_u2/2}" rpy="0 0 0"/>
+        <geometry>
+          <box size="${lx_u2} ${ly_u2} ${lz_u2}"/>
+        </geometry>
+      </collision>
+    </link>
+    <joint name="${prefix}_K0" type="revolute" >
+      <parent link="${prefix}_u2"/>
+      <child link="${prefix}_l0"/>
+      <origin xyz="0 0 ${-lz_u2}"/>
+      <axis xyz="0 1 0"/>
+      <dynamics damping="${joint_damping}" friction="${joint_friction}"/>
+      <limit effort="${joint_effort}" velocity="${joint_vel}" lower="0" upper="${7*pi/8}" />
+    </joint>
+    <transmission name="${prefix}_K0_tran">
+      <type>transmission_interface/SimpleTransmission</type>
+      <joint name="${prefix}_K0">
+        <hardwareInterface>hardware_interface/EffortJointInterface</hardwareInterface>
+      </joint>
+      <actuator name="${prefix}_K0_motor">
+        <hardwareInterface>hardware_interface/EffortJointInterface</hardwareInterface>
+        <mechanicalReduction>1</mechanicalReduction>
+      </actuator>
+    </transmission>
+    <link name="${prefix}_l0" >
+      <visual>
+        <origin xyz="0 0 ${-lz_l0/2}" rpy="0 0 0"/>
+        <geometry>
+          <box size="${lx_l0} ${ly_l0} ${lz_l0}"/>
+        </geometry>
+        <material name="orange"/>
+      </visual>
+      <inertial>
+        <origin xyz="0 0 ${-lz_l0/2}" rpy="0 0 0"/>
+        <xacro:box_inertia  lenx="${lx_l0}" leny="${ly_l0}" lenz="${lz_l0}" />
+      </inertial>
+      <collision>
+       <origin xyz="0 0 ${-lz_l0/2}" rpy="0 0 0"/>
+       <geometry>
+         <box size="${lx_l0} ${ly_l0} ${lz_l0}"/>
+       </geometry>
+      </collision>
+    </link>
+    <joint name="${prefix}_A0" type="revolute" >
+      <parent link="${prefix}_l0"/>
+      <child link="${prefix}_l1"/>
+      <origin xyz="0 0 ${-lz_l0+lz_l1/2}" rpy="0 0 0"/>
       <axis xyz="1 0 0"/>
-      <dynamics damping="0.9"/>
-      <limit effort="2" velocity="1.0" lower="${-pi/2}" upper="${pi/2}" />
-    </joint>
-    <link name="${prefix}_hip_3" >
-      <visual>
-        <origin xyz="0 0 ${-lenz_hip_3/2 }" rpy="0 0 0"/>
-        <geometry>
-          <box size="${lenx_hip_3} ${leny_hip_3} ${lenz_hip_3}"/>
+      <dynamics damping="${joint_damping}" friction="${joint_friction}"/>
+      <limit effort="${joint_effort}" velocity="${joint_vel}" lower="${-pi/4}" upper="${pi/4}" />
+    </joint>
+    <transmission name="${prefix}_A0_tran">
+      <type>transmission_interface/SimpleTransmission</type>
+      <joint name="${prefix}_A0">
+        <hardwareInterface>hardware_interface/EffortJointInterface</hardwareInterface>
+      </joint>
+      <actuator name="${prefix}_A0_motor">
+        <hardwareInterface>hardware_interface/EffortJointInterface</hardwareInterface>
+        <mechanicalReduction>1</mechanicalReduction>
+      </actuator>
+    </transmission>
+    <link name="${prefix}_l1" >
+      <visual>
+      <origin xyz="0 0 0" rpy="0 0 0"/>
+        <geometry>
+          <box size="${lx_l1} ${ly_l1} ${lz_l1}"/>
+        </geometry>
+        <material name="black"/>
+      </visual>
+      <inertial>
+        <origin xyz="0 0 0" rpy="0 0 0"/>
+        <xacro:box_inertia  lenx="${lx_l1}" leny="${ly_l1}" lenz="${lz_l1}" />
+      </inertial>
+      <collision>
+        <origin xyz="0 0 0" rpy="0 0 0"/>
+        <geometry>
+          <box size="${lx_l1} ${ly_l1} ${lz_l1}"/>
+        </geometry>
+      </collision>
+    </link>
+    <joint name="${prefix}_A1" type="revolute" >
+      <parent link="${prefix}_l1"/>
+      <child link="${prefix}_l2"/>
+      <origin xyz="${-lx_l1/2} 0 0"/>
+      <axis xyz="0 1 0"/>
+      <dynamics damping="${joint_damping}" friction="${joint_friction}"/>
+      <limit effort="${joint_effort}" velocity="${joint_vel}" lower="${-pi/4}" upper="${pi/4}" />
+    </joint>
+    <transmission name="${prefix}_A1_tran">
+      <type>transmission_interface/SimpleTransmission</type>
+      <joint name="${prefix}_A1">
+        <hardwareInterface>hardware_interface/EffortJointInterface</hardwareInterface>
+      </joint>
+      <actuator name="${prefix}_A1_motor">
+        <hardwareInterface>hardware_interface/EffortJointInterface</hardwareInterface>
+        <mechanicalReduction>1</mechanicalReduction>
+      </actuator>
+    </transmission>
+    <link name="${prefix}_l2" >
+      <visual>
+        <origin xyz="0 0 ${-lz_l2/2}" rpy="0 0 0"/>
+        <geometry>
+          <box size="${lx_l2} ${ly_l2} ${lz_l2}"/>
         </geometry>
         <material name="orange"/>
       </visual>
-     <xacro:box_inertia  lenx="${lenx_hip_3}" leny="${leny_hip_3}" lenz="${lenz_hip_3}" />
-     <collision>
-        <origin xyz="0 0 ${-1*lenz_hip_3/2 }" rpy="0 0 0"/>
-        <geometry>
-          <box size="${lenx_hip_3} ${leny_hip_3} ${lenz_hip_3}"/>
-        </geometry>
-     </collision>
-    </link>
-    <joint name="${prefix}_hip_3_joint" type="revolute" >
-      <parent link="${prefix}_hip_3"/>
-      <child link="${prefix}_upp_leg"/>
-      <origin xyz="0 0 ${-lenz_hip_3}"/>
-      <axis xyz="0 0 1"/>
-      <dynamics damping="0.9"/>
-      <limit effort="2" velocity="1.0" lower="${-pi/2}" upper="${pi/2}" />
-    </joint>
-    <link name="${prefix}_upp_leg" >
-      <visual>
-        <origin xyz="0 0 ${-lenz_upp_leg/2}" rpy="0 0 0"/>
-        <geometry>
-          <box size="${lenx_upp_leg} ${leny_upp_leg} ${lenz_upp_leg}"/>
-        </geometry>
-        <material name="black"/>
-      </visual>
-     <xacro:box_inertia  lenx="${lenx_upp_leg}" leny="${leny_upp_leg}" lenz="${lenz_upp_leg}" />
-     <collision>
-        <origin xyz="0 0 ${-lenz_upp_leg/2}" rpy="0 0 0"/>
-        <geometry>
-          <box size="${lenx_upp_leg} ${leny_upp_leg} ${lenz_upp_leg}"/>
-        </geometry>
-     </collision>
-    </link>
-    <joint name="${prefix}_knee_joint" type="revolute" >
-      <parent link="${prefix}_upp_leg"/>
-      <child link="${prefix}_low_leg"/>
-      <origin xyz="0 0 ${-lenz_upp_leg}"/>
-      <axis xyz="0 1 0"/>
-      <dynamics damping="0.9"/>
-      <limit effort="2" velocity="1.0" lower="0" upper="${7*pi/8}" />
-    </joint>
-    <link name="${prefix}_low_leg" >
-      <visual>
-        <origin xyz="0 0 ${-lenz_low_leg/2}" rpy="0 0 0"/>
-        <geometry>
-         <box size="${lenx_low_leg} ${leny_low_leg} ${lenz_low_leg}"/>
+      <inertial>
+        <origin xyz="0 0 ${-lz_l2/2}" rpy="0 0 0"/>
+        <xacro:box_inertia  lenx="${lx_l2}" leny="${ly_l2}" lenz="${lz_l2}" />
+      </inertial>
+      <collision>
+        <origin xyz="0 0 ${-lz_l2/2}" rpy="0 0 0"/>
+        <geometry>
+          <box size="${lx_l2} ${ly_l2} ${lz_l2}"/>
+        </geometry>
+      </collision>
+    </link>
+    <joint name="${prefix}_l3_fix" type="fixed" >
+      <parent link="${prefix}_l2"/>
+      <child link="${prefix}_l3"/>
+      <origin xyz="0 0 ${-lz_l2}"/>
+    </joint>
+    <link name="${prefix}_l3" >
+      <visual>
+        <origin xyz="${lx_l3/2-lx_l2/2} 0 ${-lz_l3/2}" rpy="0 0 0"/>
+        <geometry>
+          <box size="${lx_l3} ${ly_l3} ${lz_l3}"/>
         </geometry>
         <material name="orange"/>
       </visual>
-     <xacro:box_inertia  lenx="${lenx_low_leg}" leny="${leny_low_leg}" lenz="${lenz_low_leg}" />
-     <collision>
-       <origin xyz="0 0 ${-lenz_low_leg/2}" rpy="0 0 0"/>
-       <geometry>
-         <box size="${lenx_low_leg} ${leny_low_leg} ${lenz_low_leg}"/>
-       </geometry>
-     </collision>
-    </link>
-    <joint name="${prefix}_ang_1_joint" type="revolute" >
-      <parent link="${prefix}_low_leg"/>
-      <child link="${prefix}_ang_1"/>
-      <origin xyz="0 0 ${-lenz_low_leg+lenz_ang_1/2}" rpy="0 0 0"/>
-      <axis xyz="1 0 0"/>
-      <dynamics damping="0.9"/>
-      <limit effort="2" velocity="1.0" lower="${-pi/4}" upper="${pi/4}" />
-    </joint>
-    <link name="${prefix}_ang_1" >
-      <visual>
-      <origin xyz="0 0 0" rpy="0 0 0"/>
-        <geometry>
-          <box size="${lenx_ang_1} ${leny_ang_1} ${lenz_ang_1}"/>
-        </geometry>
-        <material name="black"/>
-      </visual>
-     <xacro:box_inertia  lenx="${lenx_ang_1}" leny="${leny_ang_1}" lenz="${lenz_ang_1}" />
-     <collision>
-       <origin xyz="0 0 0" rpy="0 0 0"/>
-       <geometry>
-         <box size="${lenx_ang_1} ${leny_ang_1} ${lenz_ang_1}"/>
-       </geometry>
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
File: robotv1_description/urdf/lower_body.xacro (robot description, xacro)
@@ -1,25 +1,63 @@
 <?xml version="1.0"?>
-<robot name="upper_body" xmlns:xacro="http://www.ros.org/wiki/xacro">
+<robot xmlns:xacro="http://www.ros.org/wiki/xacro">
   <xacro:include filename="$(find robotv1_description)/urdf/leg.xacro"/>
-  <xacro:property name="lenx_pelvis" value="0.08"/>
-  <xacro:property name="leny_pelvis" value="0.16"/>
-  <xacro:property name="lenz_pelvis" value="0.06"/>
+  <xacro:include filename="$(find robotv1_description)/urdf/lower_body.gazebo"/>
+  <xacro:property name="lx_pelvis" value="0.05"/>
+  <xacro:property name="ly_pelvis" value="0.10"/>
+  <xacro:property name="lz_pelvis" value="0.04"/>
+  <xacro:property name="lx_imu_link" value="0.03"/>
+  <xacro:property name="ly_imu_link" value="0.03"/>
+  <xacro:property name="lz_imu_link" value="0.005"/>
+  <xacro:property name="pos_pelvis" value="${lz_u1 + lz_u2+ lz_l0 + lz_l2/2.0 + lz_l3}"/>
+  <link name="world"/>
+  <joint name="world_to_pelvis" type="fixed">
+    <origin xyz="0 0 ${pos_pelvis+ 0.2}" rpy="0 0 0"/>
+    <parent link="world" />
+    <child link="pelvis" />
+  </joint>
   <link name="pelvis" >
     <visual>
-      <origin xyz="0 0 0 " rpy="0 0 0" />
+      <origin xyz="0 0 0" rpy="0 0 0" />
       <geometry>
-        <box size="${lenx_pelvis} ${leny_pelvis} ${lenz_pelvis}"/>
+        <box size="${lx_pelvis} ${ly_pelvis} ${lz_pelvis}"/>
       </geometry>
-      <material name="orange"/>
+      <material name="white"/>
     </visual>
-    <xacro:box_inertia lenx="${lenx_pelvis}" leny="${leny_pelvis}" lenz="${lenz_pelvis}"/>
+    <inertial>
+      <origin xyz="0 0 0" rpy="0 0 0" />
+      <xacro:box_inertia lenx="${lx_pelvis}" leny="${ly_pelvis}" lenz="${lz_pelvis}"/>
+    </inertial>
     <collision>
-      <origin xyz="0 0 0 " rpy="0 0 0" />
+      <origin xyz="0 0 0" rpy="0 0 0" />
       <geometry>
-        <box size="${lenx_pelvis} ${leny_pelvis} ${lenz_pelvis}"/>
+        <box size="${lx_pelvis} ${ly_pelvis} ${lz_pelvis}"/>
       </geometry>
     </collision>
   </link>
-  <xacro:leg prefix="left_leg" reflect="1" />
-  <xacro:leg prefix="right_leg" reflect="-1" />
+  <joint name="pelvis_to_imu_link" type="fixed">
+    <origin xyz="0 0 ${-lz_pelvis/2.0}" rpy="0 0 0" />
+    <parent link="pelvis"/>
+    <child link="imu_link_pelvis"/>
+  </joint>
+  <link name="imu_link_pelvis" >
+    <visual>
+      <origin xyz="0 0 ${-lz_imu_link/2.0}" rpy="0 0 0" />
+      <geometry>
+        <box size="${lx_imu_link} ${ly_imu_link} ${lz_imu_link}"/>
+      </geometry>
+      <material name="blue"/>
+    </visual>
+    <inertial>
+      <origin xyz="0 0 ${lz_imu_link/2.0}" rpy="0 0 0" />
+      <xacro:box_inertia lenx="${lx_imu_link}" leny="${ly_imu_link}" lenz="${lz_imu_link}"/>
+    </inertial>
+    <collision>
+      <origin xyz="0 0 0" rpy="0 0 0" />
+      <geometry>
+        <box size="${lx_imu_link} ${ly_imu_link} ${lz_imu_link}"/>
+      </geometry>
+    </collision>
+  </link>
+  <xacro:leg prefix="LLEG" reflect="1" />
+  <xacro:leg prefix="RLEG" reflect="-1" />
 </robot>

File: robotv1_description/urdf/robotv1.xacro (robot description, xacro)
@@ -1,18 +1,5 @@
 <?xml version="1.0"?>
 <robot name="robotv1" xmlns:xacro="http://www.ros.org/wiki/xacro">
-<xacro:include filename="$(find robotv1_description)/urdf/leg.xacro"/>
-<xacro:include filename="$(find robotv1_description)/urdf/arm.xacro"/>
-<xacro:include filename="$(find robotv1_description)/urdf/torso.xacro"/>
-<xacro:include filename="$(find robotv1_description)/materials/materials.xacro" />
-<!-- only gazebo plug-in -->
-<xacro:include filename="$(find robotv1_description)/urdf/robotv1.gazebo"/>
-<link name="dummy"/>
-<joint name="dummy_to_pelvis" type="fixed">
-  <origin xyz="0 0 ${base_pos}" rpy="0 0 0"/>
-  <parent link="dummy" />
-  <child link="pelvis" />
-</joint>
-<xacro:leg prefix="leftleg" reflect="1"/>
-<xacro:leg prefix="rightleg" reflect="-1"/>
-<xacro:arm prefix="leftarm" />
+<xacro:include filename="$(find robotv1_description)/materials/materials.xacro"/>
+<xacro:include filename="$(find robotv1_description)/urdf/lower_body.xacro"/>
 </robot>

File: robotv1_description/urdf/utilities.xacro (robot description, xacro)
@@ -1,14 +1,12 @@
 <?xml version="1.0"?>
 <robot xmlns:xacro="http://www.ros.org/wiki/xacro">
-  <xacro:property name="density" value="2700"/>
+  <xacro:property name="density" value="1700"/>
   <xacro:macro name="box_inertia" params="lenx leny lenz">
     <xacro:property name="mass" value="${density * lenx * leny * lenz}"/>
-    <inertial>
-      <mass value="${mass}" />
-      <inertia
+    <mass value="${mass}" />
+    <inertia
       ixx="${mass*(lenz*lenz+leny*leny)/12.0}" ixy="0.0" ixz="0.0"
       iyy="${mass*(lenz*lenz+lenx*lenx)/12.0}" iyz="0.0"
       izz="${mass*(lenx*lenx+leny*leny)/12.0}" />
-    </inertial>
   </xacro:macro>
 </robot>
