Commit message: publisher

File: robotv1_description/urdf/leg.xacro (robot description, xacro)
@@ -6,5 +6,5 @@
   <xacro:property name="joint_damping" value="0.03"/>
   <xacro:property name="joint_effort" value="10.0"/>
-  <xacro:property name="joint_vel" value="3.0"/>
+  <xacro:property name="joint_vel" value="6.0"/>
   <xacro:property name="lx_u0" value="0.04"/>
   <xacro:property name="ly_u0" value="0.03"/>
@@ -27,5 +27,8 @@
   <xacro:property name="lx_l3" value="0.1"/>
   <xacro:property name="ly_l3" value="0.04"/>
-  <xacro:property name="lz_l3" value="0.01"/>
+  <xacro:property name="lz_l3" value="0.008"/>
+  <xacro:property name="lx_l4" value="0.1"/>
+  <xacro:property name="ly_l4" value="0.04"/>
+  <xacro:property name="lz_l4" value="0.005"/>
   <xacro:property name="lx_imu_link" value="0.03"/>
   <xacro:property name="ly_imu_link" value="0.03"/>
@@ -283,4 +286,39 @@
       </collision>
     </link>
+    <joint name="${prefix}_ft_sensor" type="revolute" >
+      <parent link="${prefix}_l3"/>
+      <child link="${prefix}_l4"/>
+      <origin xyz="${lx_l4/2-lx_l2/2} 0 ${-lz_l3}"/>
+      <limit effort="10.0" velocity="1.0" upper="0.0" lower="0.0"/>
+    </joint>
+    <transmission name="${prefix}_ft_sensor_tran">
+      <type>transmission_interface/SimpleTransmission</type>
+      <joint name="${prefix}_ft_sensor">
+        <hardwareInterface>hardware_interface/EffortJointInterface</hardwareInterface>
+      </joint>
+      <actuator name="${prefix}_ft_sensor_motor">
+        <hardwareInterface>hardware_interface/EffortJointInterface</hardwareInterface>
+        <mechanicalReduction>1</mechanicalReduction>
+      </actuator>
+    </transmission>
+    <link name="${prefix}_l4" >
+      <visual>
+        <origin xyz="0 0 ${-lz_l4/2}" rpy="0 0 0"/>
+        <geometry>
+          <box size="${lx_l4} ${ly_l4} ${lz_l4}"/>
+        </geometry>
+        <material name="black"/>
+      </visual>
+      <inertial>
+        <origin xyz="0 0 ${-lz_l4/2}" rpy="0 0 0"/>
+        <xacro:box_inertia  lenx="${lx_l4}" leny="${ly_l4}" lenz="${lz_l4}" />
+      </inertial>
+      <collision>
+        <origin xyz="0 0 ${-lz_l4/2}" rpy="0 0 0"/>
+        <geometry>
+           <box size="${lx_l4} ${ly_l4} ${lz_l4}"/>
+        </geometry>
+      </collision>
+    </link>
     <joint name="${prefix}_l3_to_imu_link" type="fixed">
       <origin xyz="${lx_l3/2} 0 0" rpy="0 0 0" />

File: robotv1_description/urdf/lower_body.xacro (robot description, xacro)
@@ -10,8 +10,16 @@
   <xacro:property name="lz_imu_link" value="0.005"/>
   <xacro:property name="pos_pelvis" value="${lz_u1 + lz_u2+ lz_l0 + lz_l2/2.0 + lz_l3}"/>
+<!--
   <link name="world"/>
-  <joint name="world_to_pelvis" type="fixed">
+  <joint name="world_to_dummy" type="fixed">
+    <origin xyz="0 0 0" rpy="0 0 0"/>
+    <parent link="world" />
+    <child link="dummy" />
+  </joint>
+-->
+  <link name="dummy" />
+  <joint name="dummy_to_pelvis" type="fixed">
     <origin xyz="0 0 ${pos_pelvis+ 0.2}" rpy="0 0 0"/>
-    <parent link="world" />
+    <parent link="dummy" />
     <child link="pelvis" />
   </joint>

File: robotv1_description/urdf/robotv1.urdf (robot description, URDF)
Before this commit: robot robotv1, 19 links, 18 joints
Links:
- removed link imu_link
- removed link wolrd
- added link LLEG_l4, mass 0.034; collision box size=0.1 0.04 0.005; visual box size=0.1 0.04 0.005
- added link RLEG_l4, mass 0.034; collision box size=0.1 0.04 0.005; visual box size=0.1 0.04 0.005
- added link dummy
- added link imu_link_pelvis, mass 0.00765; collision box size=0.03 0.03 0.005; visual box size=0.03 0.03 0.005
- link LLEG_imu_link: mass 0.009 -> 0.00765
- link LLEG_l0: mass 0.072 -> 0.0612
- link LLEG_l1: mass 0.144 -> 0.1224
- link LLEG_l2: mass 0.144 -> 0.1224
- link LLEG_l3: mass 0.08 -> 0.0544; geometry collision box size=0.1 0.04 0.008; visual box size=0.1 0.04 0.008
- link LLEG_u0: mass 0.144 -> 0.1224
- link LLEG_u1: mass 0.324 -> 0.2754
- link LLEG_u2: mass 0.144 -> 0.1224
- link RLEG_imu_link: mass 0.009 -> 0.00765
- link RLEG_l0: mass 0.072 -> 0.0612
- link RLEG_l1: mass 0.144 -> 0.1224
- link RLEG_l2: mass 0.144 -> 0.1224
- link RLEG_l3: mass 0.08 -> 0.0544; geometry collision box size=0.1 0.04 0.008; visual box size=0.1 0.04 0.008
- link RLEG_u0: mass 0.144 -> 0.1224
- link RLEG_u1: mass 0.324 -> 0.2754
- link RLEG_u2: mass 0.144 -> 0.1224
- link pelvis: mass 0.4 -> 0.34
Joints:
- removed joint wolrd_to_pelvis
- added joint LLEG_ft_sensor: type fixed, parent LLEG_l3, child LLEG_l4, origin xyz=0.035 0 -0.008
- added joint RLEG_ft_sensor: type fixed, parent RLEG_l3, child RLEG_l4, origin xyz=0.035 0 -0.008
- added joint dummy_to_pelvis: type fixed, parent dummy, child pelvis, origin xyz=0 0 0.548 rpy=0 0 0
- joint LLEG_A0: limit lower=-0.785398163397 upper=0.785398163397 effort=30.0 velocity=6.28318530718 -> lower=-0.785398163397 upper=0.785398163397 effort=10.0 velocity=6.0
- joint LLEG_A1: limit lower=-0.785398163397 upper=0.785398163397 effort=30.0 velocity=6.28318530718 -> lower=-0.785398163397 upper=0.785398163397 effort=10.0 velocity=6.0
- joint LLEG_H0: limit lower=-1.57079632679 upper=1.57079632679 effort=30.0 velocity=6.28318530718 -> lower=-1.57079632679 upper=1.57079632679 effort=10.0 velocity=6.0
- joint LLEG_H1: limit lower=-1.57079632679 upper=1.57079632679 effort=30.0 velocity=6.28318530718 -> lower=-1.57079632679 upper=1.57079632679 effort=10.0 velocity=6.0
- joint LLEG_H2: limit lower=-1.57079632679 upper=1.57079632679 effort=30.0 velocity=6.28318530718 -> lower=-1.57079632679 upper=1.57079632679 effort=10.0 velocity=6.0
- joint LLEG_K0: limit lower=0 upper=2.74889357189 effort=30.0 velocity=6.28318530718 -> lower=0 upper=2.74889357189 effort=10.0 velocity=6.0
- joint RLEG_A0: limit lower=-0.785398163397 upper=0.785398163397 effort=30.0 velocity=6.28318530718 -> lower=-0.785398163397 upper=0.785398163397 effort=10.0 velocity=6.0
- joint RLEG_A1: limit lower=-0.785398163397 upper=0.785398163397 effort=30.0 velocity=6.28318530718 -> lower=-0.785398163397 upper=0.785398163397 effort=10.0 velocity=6.0
- joint RLEG_H0: limit lower=-1.57079632679 upper=1.57079632679 effort=30.0 velocity=6.28318530718 -> lower=-1.57079632679 upper=1.57079632679 effort=10.0 velocity=6.0
- joint RLEG_H1: limit lower=-1.57079632679 upper=1.57079632679 effort=30.0 velocity=6.28318530718 -> lower=-1.57079632679 upper=1.57079632679 effort=10.0 velocity=6.0
- joint RLEG_H2: limit lower=-1.57079632679 upper=1.57079632679 effort=30.0 velocity=6.28318530718 -> lower=-1.57079632679 upper=1.57079632679 effort=10.0 velocity=6.0
- joint RLEG_K0: limit lower=0 upper=2.74889357189 effort=30.0 velocity=6.28318530718 -> lower=0 upper=2.74889357189 effort=10.0 velocity=6.0
- joint pelvis_to_imu_link: child imu_link -> imu_link_pelvis

Commit message: add features

File: robotv1_description/urdf/leg.xacro (robot description, xacro)
@@ -12,22 +12,22 @@
   <xacro:property name="lx_u1" value="0.06"/>
   <xacro:property name="ly_u1" value="0.03"/>
-  <xacro:property name="lz_u1" value="0.09"/>
+  <xacro:property name="lz_u1" value="0.08"/>
   <xacro:property name="lx_u2" value="0.03"/>
   <xacro:property name="ly_u2" value="0.04"/>
-  <xacro:property name="lz_u2" value="0.06"/>
+  <xacro:property name="lz_u2" value="0.08"/>
   <xacro:property name="lx_l0" value="0.015"/>
   <xacro:property name="ly_l0" value="0.015"/>
-  <xacro:property name="lz_l0" value="0.16"/>
+  <xacro:property name="lz_l0" value="0.13"/>
   <xacro:property name="lx_l1" value="0.04"/>
   <xacro:property name="ly_l1" value="0.03"/>
-  <xacro:property name="lz_l1" value="0.06"/>
-  <xacro:property name="lx_l2" value="0.03"/>
+  <xacro:property name="lz_l1" value="0.04"/>
+  <xacro:property name="lx_l2" value="0.02"/>
   <xacro:property name="ly_l2" value="0.04"/>
-  <xacro:property name="lz_l2" value="0.06"/>
-  <xacro:property name="lx_l3" value="0.1"/>
-  <xacro:property name="ly_l3" value="0.04"/>
+  <xacro:property name="lz_l2" value="0.02"/>
+  <xacro:property name="lx_l3" value="0.12"/>
+  <xacro:property name="ly_l3" value="0.05"/>
   <xacro:property name="lz_l3" value="0.008"/>
-  <xacro:property name="lx_l4" value="0.1"/>
-  <xacro:property name="ly_l4" value="0.04"/>
+  <xacro:property name="lx_l4" value="0.12"/>
+  <xacro:property name="ly_l4" value="0.05"/>
   <xacro:property name="lz_l4" value="0.005"/>
   <xacro:property name="lx_imu_link" value="0.03"/>
@@ -83,5 +83,5 @@
        <axis xyz="1 0 0"/>
        <dynamics damping="${joint_damping}" friction="${joint_friction}"/>
-       <limit effort="${joint_effort}" velocity="${joint_vel}" lower="${-pi/2}" upper="${pi/2}" />
+       <limit effort="${joint_effort}" velocity="${joint_vel}" lower="${-pi/4}" upper="${pi/4}" />
     </joint>
     <transmission name="${prefix}_H1_tran">
@@ -101,5 +101,5 @@
           <box size="${lx_u1} ${ly_u1} ${lz_u1}"/>
         </geometry>
-        <material name="orange"/>
+        <material name="white"/>
       </visual>
       <inertial>
@@ -120,5 +120,5 @@
       <axis xyz="0 0 1"/>
       <dynamics damping="${joint_damping}" friction="${joint_friction}"/>
-      <limit effort="${joint_effort}" velocity="${joint_vel}" lower="${-pi/2}" upper="${pi/2}" />
+      <limit effort="${joint_effort}" velocity="${joint_vel}" lower="${-pi/4}" upper="${pi/4}" />
     </joint>
     <transmission name="${prefix}_H2_tran">
@@ -175,5 +175,5 @@
           <box size="${lx_l0} ${ly_l0} ${lz_l0}"/>
         </geometry>
-        <material name="orange"/>
+        <material name="white"/>
       </visual>
       <inertial>
@@ -191,8 +191,8 @@
       <parent link="${prefix}_l0"/>
       <child link="${prefix}_l1"/>
-      <origin xyz="0 0 ${-lz_l0+lz_l1/2}" rpy="0 0 0"/>
-      <axis xyz="1 0 0"/>
-      <dynamics damping="${joint_damping}" friction="${joint_friction}"/>
-      <limit effort="${joint_effort}" velocity="${joint_vel}" lower="${-pi/4}" upper="${pi/4}" />
+      <origin xyz="0 0 ${-lz_l0}" rpy="0 0 0"/>
+      <axis xyz="0 1 0"/>
+      <dynamics damping="${joint_damping}" friction="${joint_friction}"/>
+      <limit effort="${joint_effort}" velocity="${joint_vel}" lower="${-pi/2}" upper="${pi/2}" />
     </joint>
     <transmission name="${prefix}_A0_tran">
@@ -208,5 +208,5 @@
     <link name="${prefix}_l1" >
       <visual>
-      <origin xyz="0 0 0" rpy="0 0 0"/>
+      <origin xyz="0 0 ${-lz_l1/2}" rpy="0 0 0"/>
         <geometry>
           <box size="${lx_l1} ${ly_l1} ${lz_l1}"/>
@@ -215,9 +215,9 @@
       </visual>
       <inertial>
-        <origin xyz="0 0 0" rpy="0 0 0"/>
+        <origin xyz="0 0 ${-lz_l1/2}" rpy="0 0 0"/>
         <xacro:box_inertia  lenx="${lx_l1}" leny="${ly_l1}" lenz="${lz_l1}" />
       </inertial>
       <collision>
-        <origin xyz="0 0 0" rpy="0 0 0"/>
+        <origin xyz="0 0 ${-lz_l1/2}" rpy="0 0 0"/>
         <geometry>
           <box size="${lx_l1} ${ly_l1} ${lz_l1}"/>
@@ -228,6 +228,6 @@
       <parent link="${prefix}_l1"/>
       <child link="${prefix}_l2"/>
-      <origin xyz="${-lx_l1/2} 0 0"/>
-      <axis xyz="0 1 0"/>
+      <origin xyz="0 0 ${-lz_l1}"/>
+      <axis xyz="1 0 0"/>
       <dynamics damping="${joint_damping}" friction="${joint_friction}"/>
       <limit effort="${joint_effort}" velocity="${joint_vel}" lower="${-pi/4}" upper="${pi/4}" />
@@ -245,16 +245,16 @@
     <link name="${prefix}_l2" >
       <visual>
-        <origin xyz="0 0 ${-lz_l2/2}" rpy="0 0 0"/>
+        <origin xyz="0 0 0" rpy="0 0 0"/>
         <geometry>
           <box size="${lx_l2} ${ly_l2} ${lz_l2}"/>
         </geometry>
-        <material name="orange"/>
-      </visual>
-      <inertial>
-        <origin xyz="0 0 ${-lz_l2/2}" rpy="0 0 0"/>
+        <material name="white"/>
+      </visual>
+      <inertial>
+        <origin xyz="0 0 0" rpy="0 0 0"/>
         <xacro:box_inertia  lenx="${lx_l2}" leny="${ly_l2}" lenz="${lz_l2}" />
       </inertial>
       <collision>
-        <origin xyz="0 0 ${-lz_l2/2}" rpy="0 0 0"/>
+        <origin xyz="0 0 0" rpy="0 0 0"/>
         <geometry>
           <box size="${lx_l2} ${ly_l2} ${lz_l2}"/>
@@ -265,20 +265,20 @@
       <parent link="${prefix}_l2"/>
       <child link="${prefix}_l3"/>
-      <origin xyz="0 0 ${-lz_l2}"/>
+      <origin xyz="${lx_l2/4} 0 ${-lz_l2/2}"/>
     </joint>
     <link name="${prefix}_l3" >
       <visual>
-        <origin xyz="${lx_l3/2-lx_l2/2} 0 ${-lz_l3/2}" rpy="0 0 0"/>
+        <origin xyz="0 0 ${-lz_l3/2}" rpy="0 0 0"/>
         <geometry>
           <box size="${lx_l3} ${ly_l3} ${lz_l3}"/>
         </geometry>
-        <material name="orange"/>
-      </visual>
-      <inertial>
-        <origin xyz="${lx_l3/2-lx_l2/2} 0 ${-lz_l3/2}" rpy="0 0 0"/>
+        <material name="white"/>
+      </visual>
+      <inertial>
+        <origin xyz="0 0 ${-lz_l3/2}" rpy="0 0 0"/>
         <xacro:box_inertia  lenx="${lx_l3}" leny="${ly_l3}" lenz="${lz_l3}" />
       </inertial>
       <collision>
-        <origin xyz="${lx_l3/2-lx_l2/2} 0 ${-lz_l3/2}" rpy="0 0 0"/>
+        <origin xyz="0 0 ${-lz_l3/2}" rpy="0 0 0"/>
         <geometry>
            <box size="${lx_l3} ${ly_l3} ${lz_l3}"/>
@@ -289,5 +289,5 @@
       <parent link="${prefix}_l3"/>
       <child link="${prefix}_l4"/>
-      <origin xyz="${lx_l4/2-lx_l2/2} 0 ${-lz_l3}"/>
+      <origin xyz="0 0 ${-lz_l3}"/>
       <limit effort="10.0" velocity="1.0" upper="0.0" lower="0.0"/>
     </joint>
@@ -322,5 +322,5 @@
     </link>
     <joint name="${prefix}_l3_to_imu_link" type="fixed">
-      <origin xyz="${lx_l3/2} 0 0" rpy="0 0 0" />
+      <origin xyz="${lx_l3/2-lx_imu_link/2} 0 0" rpy="0 0 0" />
       <parent link="${prefix}_l3"/>
       <child link="${prefix}_imu_link"/>

File: robotv1_description/urdf/lower_body.xacro (robot description, xacro)
@@ -9,5 +9,5 @@
   <xacro:property name="ly_imu_link" value="0.03"/>
   <xacro:property name="lz_imu_link" value="0.005"/>
-  <xacro:property name="pos_pelvis" value="${lz_u1 + lz_u2+ lz_l0 + lz_l2/2.0 + lz_l3}"/>
+  <xacro:property name="pos_pelvis" value="${lz_u1 + lz_u2+ lz_l0 + lz_l1 + lz_l2/2 + lz_l3 + lz_l4}"/>
 <!--
   <link name="world"/>
@@ -20,5 +20,5 @@
   <link name="dummy" />
   <joint name="dummy_to_pelvis" type="fixed">
-    <origin xyz="0 0 ${pos_pelvis+ 0.2}" rpy="0 0 0"/>
+    <origin xyz="0 0 ${pos_pelvis}" rpy="0 0 0"/>
     <parent link="dummy" />
     <child link="pelvis" />
